File: lv/bruno-white/bruno-white.kicad_sch (KiCad schematic)
At the start: 6 parts, among them U1 INA128

Commit message: LV and PE edits
Assigned footprints to my strain gauge to make a PCB design, but then apparently they aren't connected so I need to fix that... I gave up on my strain gauge pcb and then for PE I was just messing around with the PCB design which worked for my buck converter. I have also added the link to my google docs!!!
Parts:
- R1, R2: footprint (none) -> Resistor_SMD:R_0603_1608Metric_Pad0.98x0.95mm_HandSolder
- Rg1: renamed from Rg; footprint (none) -> Resistor_SMD:R_0603_1608Metric_Pad0.98x0.95mm_HandSolder
- SG1: renamed from SG; footprint (none) -> Connector_Wire:SolderWire-0.1sqmm_1x01_D0.4mm_OD1mm
- renumbered SG to SG2
Changed lines of the file:
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@@
 		(in_pos_files yes)
 		(dnp no)
-		(property "Reference" "Rg"
+		(property "Reference" "Rg1"
 			(at 160.02 66.0399 0)
 			(show_name no)
@@
 			)
 		)
-		(property "Footprint" ""
+		(property "Footprint" "Resistor_SMD:R_0603_1608Metric_Pad0.98x0.95mm_HandSolder"
 			(at 162.56 67.31 0)
 			(hide yes)
@@
 			(project "bruno-white"
 				(path "/e994741c-7c7d-4124-9d00-43b883baa61d"
-					(reference "Rg")
+					(reference "Rg1")
 					(unit 1)
 				)
@@
 			)
 		)
-		(property "Footprint" ""
+		(property "Footprint" "Resistor_SMD:R_0603_1608Metric_Pad0.98x0.95mm_HandSolder"
 			(at 105.41 62.23 0)
 			(hide yes)
@@
 		(in_pos_files yes)
 		(dnp no)
-		(property "Reference" "SG"
+		(property "Reference" "SG2"
 			(at 119.38 72.3899 0)
 			(show_name no)
@@
 			(project "bruno-white"
 				(path "/e994741c-7c7d-4124-9d00-43b883baa61d"
-					(reference "SG")
+					(reference "SG2")
 					(unit 1)
 				)
@@
 			)
 		)
-		(property "Footprint" ""
+		(property "Footprint" "Resistor_SMD:R_0603_1608Metric_Pad0.98x0.95mm_HandSolder"
 			(at 105.41 73.66 0)
 			(hide yes)
@@
 		(in_pos_files yes)
 		(dnp no)
-		(property "Reference" "SG"
+		(property "Reference" "SG1"
 			(at 119.38 60.9599 0)
 			(show_name no)
@@
 			)
 		)
-		(property "Footprint" ""
+		(property "Footprint" "Connector_Wire:SolderWire-0.1sqmm_1x01_D0.4mm_OD1mm"
 			(at 116.84 62.23 0)
 			(hide yes)
@@
 			(project "bruno-white"
 				(path "/e994741c-7c7d-4124-9d00-43b883baa61d"
-					(reference "SG")
-					(unit 1)
-				)
+					(reference "SG1")
+					(unit 1)
+				)
