File: lv/kicad tut/template.kicad_sch (KiCad schematic)
At the start: 0 parts

Commit message: part 1
Parts:
- added C1: C, symbol Device:C
- added J1: Conn_01x02, symbol Connector_Generic:Conn_01x02
- added U1: MCP6004, Package_SO:SOIC-14_3.9x8.7mm_P1.27mm, symbol Amplifier_Operational:MCP6004
Connections:
- new net: C1.1, U1.1, U1.2 (-)
- new net GND: C1.2
- new net wire: J1.1 (Pin_1), J1.2 (Pin_2), U1.3 (+)
- no-connect marks 0 -> 1
