File: lv/Kicad Projects/FINAL FPC Strain Gauge/FPC Strain Gauge Circuit/FPC Strain Gauge Circuit.kicad_pcb (KiCad board)
At the start: 4 copper layers, 23 x 10 mm, 27 parts, among them U1 INA333xxDGK, U2 OPA333xxDBV, U3 ADS1220IRVAR

Commit message: Finish Kicad Strain Gauge Design and Create a readme explaining it all
Finished FPC Strain Gauge
Routing:
- added copper zone on In2.Cu, net +3V3_A
- added copper zone on In1.Cu, net AGND
Changed lines of the file:
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@@
 	(layers
 		(0 "F.Cu" signal "Signal_Top")
-		(4 "In1.Cu" power "GND")
-		(6 "In2.Cu" power "3V3")
+		(4 "In1.Cu" power "AGND")
+		(6 "In2.Cu" power "3V3_A")
 		(2 "B.Cu" signal "Signal_Bottom")
 		(9 "F.Adhes" user "F.Adhesive")
@@
 		(capping no)
 		(filling no)
+		(zone_defaults)
 		(pcbplotparams
 			(layerselection 0x00000000_00000000_55555555_57555555)
@@
 		(net "Net-(R10-Pad1)")
 	)
+	(zone
+		(net "AGND")
+		(layer "In1.Cu")
+		(name "GND")
+		(hatch edge 0.5)
+		(connect_pads
+			(clearance 0.508)
+		)
+		(min_thickness 0.25)
+		(fill
+			(thermal_gap 0.5)
+			(thermal_bridge_width 0.5)
+			(island_removal_mode 0)
+		)
+		(polygon
+			(pts
+				(xy 120.379 66.679) (xy 120.396 76.679) (xy 143.379 76.679) (xy 143.379 66.679)
+			)
+		)
+	)
+	(zone
+		(net "+3V3_A")
+		(layer "In2.Cu")
+		(name "PWR")
+		(hatch edge 0.5)
+		(priority 1)
+		(connect_pads
+			(clearance 0.508)
+		)
+		(min_thickness 0.25)
+		(fill
+			(thermal_gap 0.5)
+			(thermal_bridge_width 0.5)
+			(island_removal_mode 0)
+		)
+		(polygon
+			(pts
+				(xy 120.379 76.679) (xy 143.379 76.679) (xy 143.379 66.679) (xy 120.379 66.679)
+			)
+		)
+	)
 	(embedded_fonts no)
