File: fs-5-schematics.kicad_pcb (KiCad board)
At the start: 2 copper layers, 34 x 36.8 mm, 13 parts, among them J1 12V, J2 5V, U1 TPS54202DDC

Commit message: final pcb and schm READY
Parts:
- moved Cb 3.50 mm to (86.8, 51.2), turned to -90 degrees
- renumbered Cdecoupling1 to Cd
Routing:
- net Net-(U1-SW): track 17.6 -> 10.1 mm
- net +12V: track 39.0 -> 34.7 mm
- net Net-(U1-BOOT): track 1.81 -> 4.96 mm
Other:
- board text added: "12V to 5V Buck Converter PCB Designed by Khoa Nguyen 2026-10-15"
Changed lines of the file:
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@@
 		(capping no)
 		(filling no)
-		(zone_defaults)
 		(pcbplotparams
 			(layerselection 0x00000000_00000000_55555555_5755f5ff)
@@
 		(tags "resistor handsolder")
 		(property "Reference" "R4"
-			(at -1.3 1.5 0)
+			(at -3.15 -0.05 0)
 			(layer "F.SilkS")
 			(effects
@@
 		(tags "SOT TO_SOT_SMD")
 		(property "Reference" "U1"
-			(at -3 -1.25 0)
+			(at 1.9 -2.2 0)
 			(layer "F.SilkS")
 			(effects
@@
 		(tags "capacitor handsolder")
 		(property "Reference" "Cout1"
-			(at 0 -1.68 90)
+			(at 4.25 -0.2 90)
 			(layer "F.SilkS")
-			(hide yes)
 			(effects
 				(font
-					(size 1 1)
-					(thickness 0.15)
+					(size 1.016 1.016)
+					(thickness 0.1524)
 				)
 			)
@@
 		(tags "capacitor handsolder")
 		(property "Reference" "Cout2"
-			(at 0 -1.68 90)
+			(at 4.35 0 90)
 			(layer "F.SilkS")
-			(hide yes)
 			(effects
 				(font
-					(size 1 1)
-					(thickness 0.15)
+					(size 1.016 1.016)
+					(thickness 0.1524)
 				)
 			)
@@
 		(at 79.5 51.5 -90)
 		(property "Reference" "L1"
-			(at -1 -4 0)
+			(at 0.65 -3.7 0)
 			(layer "F.SilkS")
 			(effects
@@
 		(descr "Capacitor SMD 0603 (1608 Metric), square (rectangular) end terminal, IPC-7351 nominal with elongated pad for handsoldering. (Body size source: IPC-SM-782 page 76, https://www.pcb-3d.com/wordpress/wp-content/uploads/ipc-sm-782a_amendment_1_and_2.pdf)")
 		(tags "capacitor handsolder")
-		(property "Reference" "Cdecoupling1"
-			(at -0.225 2.5 90)
+		(property "Reference" "Cd"
+			(at -0.4625 2.8 180)
 			(layer "F.SilkS")
-			(hide yes)
 			(effects
 				(font
-					(size 0.5 0.5)
-					(thickness 0.125)
+					(size 1.016 1.016)
+					(thickness 0.1524)
 				)
 			)
@@
 		(tags "resistor handsolder")
 		(property "Reference" "R3"
-			(at 2.9125 0 0)
+			(at 3.8125 0.3 0)
 			(layer "F.SilkS")
 			(effects
@@
 		(tags "capacitor handsolder")
 		(property "Reference" "Ci"
-			(at 2.9625 -1 180)
+			(at 2.7625 -0.9 180)
 			(layer "F.SilkS")
 			(effects
@@
 		(tags "resistor handsolder")
 		(property "Reference" "R2"
-			(at -2.9125 0 0)
+			(at -3.3125 -0.1 0)
 			(layer "F.SilkS")
 			(effects
@@
 	(footprint "Capacitor_SMD:C_0603_1608Metric_Pad1.08x0.95mm_HandSolder"
 		(layer "F.Cu")
-		(at 90 49.75 180)
+		(at 86.8 51.1625 -90)
 		(descr "Capacitor SMD 0603 (1608 Metric), square (rectangular) end terminal, IPC-7351 nominal with elongated pad for handsoldering. (Body size source: IPC-SM-782 page 76, https://www.pcb-3d.com/wordpress/wp-content/uploads/ipc-sm-782a_amendment_1_and_2.pdf)")
 		(tags "capacitor handsolder")
 		(property "Reference" "Cb"
-			(at 0 2.25 0)
+			(at -0.3125 1.65 180)
 			(layer "F.SilkS")
 			(effects
@@
 		)
 		(property "Value" "0.1uF"
-			(at 0 1.43 0)
+			(at 0 1.43 90)
 			(layer "F.Fab")
 			(hide yes)
@@
 		)
 		(property "Datasheet" "https://yageogroup.com/content/datasheet/asset/file/KEM_C1002_X7R_SMD"
-			(at 0 0 0)
+			(at 0 0 90)
 			(layer "F.Fab")
 			(hide yes)
@@
 		)
 		(property "Description" "Boost Capacitor 0.1 µF ±10% 16V Ceramic Capacitor X7R 0603 (1608 Metric)"
-			(at 0 0 0)
+			(at 0 0 90)
 			(layer "F.Fab")
 			(hide yes)
@@
 		)
 		(property "KiLib_Generator" "SMD_2terminal_chip_molded"
-			(at 0 0 0)
+			(at 0 0 90)
 			(layer "F.SilkS")
 			(hide yes)
@@
 		)
 		(property "Digikey Part Number" "399-17393-1-ND"
-			(at 0 0 180)
+			(at 0 0 270)
 			(unlocked yes)
 			(layer "F.Fab")
@@
 		)
 		(property "Digikey URL" "https://www.digikey.com/en/products/detail/kemet/C0603C104K4RAC7411/6873866?s=N4IgTCBcDaIMIAYBsCDMcCMCAsBpbASgIJwDs2GGIAugL5A"
-			(at 0 0 180)
+			(at 0 0 270)
 			(unlocked yes)
 			(layer "F.Fab")
@@
 		)
 		(property "Manufacturer" "KEMET"
-			(at 0 0 180)
+			(at 0 0 270)
 			(unlocked yes)
 			(layer "F.Fab")
@@
 		)
 		(property "Manufacturer Part Number" ""
-			(at 0 0 180)
+			(at 0 0 270)
 			(unlocked yes)
 			(layer "F.Fab")
@@
 		)
 		(pad "1" smd roundrect
-			(at -0.8625 0 180)
+			(at -0.8625 0 270)
 			(size 1.075 0.95)
 			(layers "F.Cu" "F.Mask" "F.Paste")
@@
 		)
 		(pad "2" smd roundrect
-			(at 0.8625 0 180)
+			(at 0.8625 0 270)
 			(size 1.075 0.95)
 			(layers "F.Cu" "F.Mask" "F.Paste")
@@
 	)
 	(gr_text "Cff"
-		(at 97 55.5 0)
+		(at 97.5 55.35 0)
 		(layer "F.SilkS")
 		(effects
@@
 		)
 	)
-	(segment
-		(start 98 52)
-		(end 98.5 52.5)
-		(width 0.254)
-		(layer "F.Cu")
-		(net "+12V")
-	)
-	(segment
-		(start 98.5 57.5)
-		(end 98 58)
-		(width 0.254)
-		(layer "F.Cu")
-		(net "+12V")
+	(gr_text "12V to 5V Buck Converter PCB\nDesigned by Khoa Nguyen\n2026-10-15"
+		(at 68.45 79.3 0)
+		(layer "F.SilkS")
+		(effects
+			(font
+				(size 1.524 1.524)
+				(thickness 0.381)
+				(bold yes)
+			)
+			(justify left bottom)
+		)
 	)
 	(segment
@@
 	)
 	(segment
-		(start 98 58)
-		(end 92 58)
+		(start 96.05 56.151974)
+		(end 96.635 56.736974)
 		(width 0.254)
 		(layer "F.Cu")
@@
 	)
 	(segment
+		(start 95.85 58.05)
+		(end 92.05 58.05)
+		(width 0.254)
+		(layer "F.Cu")
+		(net "+12V")
+	)
+	(segment
 		(start 88.8625 53.2)
 		(end 88.8625 54.2875)
@@
 	)
 	(segment
-		(start 98.5 52.5)
-		(end 98.5 57.5)
+		(start 96.05 52.65)
+		(end 96.05 56.151974)
+		(width 0.254)
+		(layer "F.Cu")
+		(net "+12V")
+	)
+	(segment
+		(start 95.4 52)
+		(end 96.05 52.65)
 		(width 0.254)
 		(layer "F.Cu")
@@
 	)
 	(segment
+		(start 96.635 56.736974)
+		(end 96.635 57.265)
+		(width 0.254)
+		(layer "F.Cu")
+		(net "+12V")
+	)
+	(segment
 		(start 88 55.15)
 		(end 87.525 55.15)
@@
 	)
 	(segment
-		(start 95.1125 52)
-		(end 98 52)
+		(start 92.05 58.05)
+		(end 92 58)
 		(width 0.254)
 		(layer "F.Cu")
@@
 	)
 	(segment
+		(start 96.635 57.265)
+		(end 95.85 58.05)
+		(width 0.254)
+		(layer "F.Cu")
+		(net "+12V")
+	)
+	(segment
+		(start 95.1125 52)
+		(end 95.4 52)
+		(width 0.254)
+		(layer "F.Cu")
+		(net "+12V")
+	)
+	(segment
 		(start 88.8625 51.3)
 		(end 88.2 51.3)
@@
 	)
 	(segment
-		(start 89.1375 49.75)
-		(end 85.75 49.75)
-		(width 0.508)
-		(layer "F.Cu")
-		(net "Net-(U1-SW)")
-	)
-	(segment
 		(start 85.104 53.92)
 		(end 79.5 53.92)
@@
 	)
 	(segment
-		(start 85.75 49.75)
-		(end 85 50.5)
-		(width 0.508)
-		(layer "F.Cu")
-		(net "Net-(U1-SW)")
-	)
-	(segment
-		(start 85 50.5)
-		(end 85 51.5)
-		(width 0.508)
-		(layer "F.Cu")
-		(net "Net-(U1-SW)")
-	)
-	(segment
 		(start 88.21529 52.25)
 		(end 88.8625 52.25)
@@
 	)
 	(segment
-		(start 85 51.5)
-		(end 85.762 52.262)
-		(width 0.508)
-		(layer "F.Cu")
-		(net "Net-(U1-SW)")
-	)
-	(segment
 		(start 88 52.262)
 		(end 86.762 52.262)
@@
 	)
 	(segment
-		(start 85.762 52.262)
-		(end 86.762 52.262)
-		(width 0.508)
-		(layer "F.Cu")
-		(net "Net-(U1-SW)")
-	)
-	(segment
 		(start 93.175 53.5)
 		(end 93.175 55.225)
@@
 	)
 	(segment
-		(start 91.1125 49.75)
-		(end 91.1375 49.775)
+		(start 91.1375 51.3)
+		(end 89.5875 49.75)
 		(width 0.254)
 		(layer "F.Cu")
@@
 	)
 	(segment
-		(start 91.1375 49.775)
-		(end 91.1375 51.3)
+		(start 89.5875 49.75)
+		(end 87.425 49.75)
 		(width 0.254)
 		(layer "F.Cu")
@@
 	)
 	(segment
-		(start 90.8625 49.75)
-		(end 91.1125 49.75)
+		(start 87 50.175)
+		(end 87.425 49.75)
 		(width 0.254)
 		(layer "F.Cu")
