File: fs-5-schematics.kicad_sch (KiCad schematic)
At the start: 13 parts, among them J1 12V, J2 5V, U1 TPS54202DDC

Commit message: final pcb and schm READY
Parts:
- L1: footprint ts-schematics:INDM5752X300N -> Project_parts:INDM5752X300N
Other:
- note added: "12V to 5V Buck Converter Drawn by Khoa Nguyen 2026-10-15"
- moved on the sheet: Cboost1, Cdecoupling1, Cfeedfoward1, Cinput1, Cout1, Cout2, J1, J2, L1, R2, R3, R4
