File: Op-Amp Based Comparator/Op-Amp Based Comparator.kicad_sch (KiCad schematic)
At the start: 11 parts, among them J1 From Brake Pressure Sensor, J2 From Current Sensor, K1 Relay_SPST-NO, U1 AD8001AN, U2 AD8001AN, U3 74LVC2G08, U4 AD8001AN

Commit message: added RC timing logic
Parts:
- added C1: 10, Package_SO:SOIC-8_3.9x4.9mm_P1.27mm, symbol Device:C
- added D1: D, symbol Device:D
- added R4: 10k, Package_DIP:DIP-8_W7.62mm, symbol Device:R
- added R5: 10k, symbol Device:R
- added R6: 144.3, Package_DIP:DIP-8_W7.62mm, symbol Device:R
- added R7: 10, Package_DIP:DIP-8_W7.62mm, symbol Device:R
- added U5: AD8001AN, Package_DIP:DIP-8_W7.62mm, symbol Amplifier_Operational:AD8001AN
Connections:
- net GND: now also K1.A2, C1.2, R5.2, U5.4 (V-)
- net at U2.2 (-): now also R2.2, R3.1
- net at K1.A1: now also R7.2
- net at U3.7: now also D1.1 (K), R4.1, R6.1, U5.7 (V+)
- new net: C1.1, D1.2 (A), R6.2, U5.3 (+)
- new net: R4.2, R5.1, U5.2 (-)
- new net: R7.1, U5.6
Other:
- note added: "~1 Second Delay Logic"
- moved on the sheet: K1, U3A
