File: lv/Aaron_BSPD/Aaron_BSPD.kicad_sch (KiCad schematic)
At the start: 0 parts

Commit message: added sensor filter and relay diode
Parts:
- added C1, C2, C3, C4, C5, C6: 0.1uF, Package_SO:SOIC-14_3.9x8.7mm_P1.27mm, symbol Device:C_Small
- added C7, C8, C9: 1F, Package_SO:SOIC-14_3.9x8.7mm_P1.27mm, symbol Device:C_Small
- added D1: D_Small, Package_TO_SOT_SMD:SOT-223-3_TabPin2, symbol Device:D_Small
- added J1: Conn_01x12_Pin, symbol Connector:Conn_01x12_Pin
- added K1: Relay_SPST-NO, Relay_THT:Relay_SPST_Omron_G5NB, symbol Relay:Relay_SPST-NO
- added Q1: BUK7880-55A, Package_TO_SOT_SMD:SOT-223-3_TabPin2, symbol Transistor_FET:BUK7880-55A
- added R1: 30K, Package_DIP:DIP-8_W7.62mm, symbol Device:R_Small
- added R10, R11, R12: 1K, Resistor_THT:R_Array_SIP4, symbol Device:R_Small
- added R2, R4, R6: 10K, symbol Device:R_Small
- added R3, R5: 124K, Package_DIP:DIP-8_W7.62mm, symbol Device:R_Small
- added R7: 35K, symbol Device:R_Small
- added R8: 23K, symbol Device:R_Small
- added R9: 2K, symbol Device:R_Small
- added U1: MCP6004, Package_DIP:DIP-14_W7.62mm_LongPads, symbol Amplifier_Operational:MCP6004
- added U2, U5, U6: MCP6004, symbol Amplifier_Operational:MCP6004
- added U3: SN74HCS08DR, Package_SO:SOIC-14_3.9x8.7mm_P1.27mm, symbol formula_slug_symbol_library:SN74HCS08DR
- added U7, U8: SN74HCS32DR, Package_SO:SOIC-14_3.9x8.7mm_P1.27mm, symbol formula_slug_symbol_library:SN74HCS32DR
Connections:
- new net: C8.1, R11.2, U1.5 (+)
- new net: C7.1, R10.2, U1.3 (+)
- new net: C9.1, R12.2, U1.10 (+)
- new net: D1.2 (A), K1.A2, Q1.2 (D)
- new net +12V: C1.1, C2.1, C3.1, C4.1, C5.1, C6.1, D1.1 (K), J1.1 (Pin_1), K1.A1, R1.1, R3.1, R5.1, R7.1, U1.4 (V+), U2.4 (V+), U3.14 (VCC), U5.4 (V+), U6.4 (V+), U7.14 (VCC)
- new net BRAKE_CHECK: U3.1, U8.3
- new net BRAKE_CURRENT_CHECK: U3.3, U8.13
- new net BRAKE_FAULT: U8.12, U8.6, U8.8, U8.9
- new net CHECK_FAULT: Q1.1 (G), U8.11
- new net CURRENT_BUFFERED: U1.1, U1.2 (-), U2.3 (+), U5.3 (+), U5.5 (+)
- new net CURRENT_CHECK: U2.1, U3.2
- new net CURRENT_FAULT: U7.3, U8.10
- new net CURRENT_OPEN: U5.7, U7.2
- new net CURRENT_SENSOR: J1.3 (Pin_3), R10.1
- new net CURRENT_SHORT: U5.1, U7.1
- new net CURRENT_VREF: R1.2, R2.1, U2.2 (-)
- new net FRONT_BRAKE_BUFFERED: U1.6 (-), U1.7, U2.5 (+), U5.10 (+), U5.12 (+)
- new net FRONT_BRAKE_CHECK: U2.7, U8.1
- new net FRONT_BRAKE_FAULT: U7.6, U8.5
- new net FRONT_BRAKE_OPEN: U5.14, U7.5
- new net FRONT_BRAKE_SENSOR: J1.4 (Pin_4), R11.1
- new net FRONT_BRAKE_SHORT: U5.8, U7.4
- new net FRONT_BRAKE_VREF: R3.2, R4.1, U2.6 (-)
- new net GND: C1.2, C2.2, C3.2, C4.2, C5.2, C6.2, C7.2, C8.2, C9.2, J1.2 (Pin_2), Q1.3 (S), R2.2, R4.2, R6.2, R9.2, U1.11 (V-), U2.11 (V-), U3.7 (GND), U5.11 (V-), U6.11 (V-), U7.7 (GND)
- new net OPEN_THRESHOLD: R8.2, R9.1, U5.13 (-), U5.6 (-), U6.6 (-)
- new net REAR_BRAKE_BUFFERED: U1.8, U1.9 (-), U2.10 (+), U6.3 (+), U6.5 (+)
- new net REAR_BRAKE_CHECK: U2.8, U8.2
- new net REAR_BRAKE_FAULT: U7.8, U8.4
- new net REAR_BRAKE_OPEN: U6.7, U7.10
- new net REAR_BRAKE_SENSOR: J1.5 (Pin_5), R12.1
- new net REAR_BRAKE_SHORT: U6.1, U7.9
- new net REAR_BRAKE_VREF: R5.2, R6.1, U2.9 (-)
- new net SHORT_THRESHOLD: R7.2, R8.1, U5.2 (-), U5.9 (-), U6.2 (-)
- new net SHUTDOWN_IN: J1.6 (Pin_6), K1.13
- new net SHUTDOWN_OUT: J1.7 (Pin_7), K1.14
- no-connect marks 0 -> 23
Other:
- note added: ".4V"
- note added: "0.9V"
- note added: "3V"
- note added: "5V"
- note added: "Aaron Mello"
- note added: "BUFFER ZONE"
- note added: "COMPARISONS"
- note added: "IF VREF(0.9V)<FRONT_BRAKE_BUFFERED then REAR_BREAK_OPEN will be high"
- note added: "IF VREF(0.9V)<REAR_BRAKE_BUFFERED then REAR_BREAK_OPEN will be high"
- note added: "IF VREF(3V)<CURRENT_BUFFERED then CURRENT_OPEN will be high"
- note added: "LOGIC"
- note added: "OPEN AND SHORT FAULTS"
- note added: "POWER"
- note added: "RELAY"
