File: pe/kicad-template/template.kicad_pcb (KiCad board)
At the start: 2 copper layers, 3 parts

Commit message: Updated schematic
Parts:
- added C2: 1uF, Capacitor_SMD:C_0603_1608Metric, F.Cu at (146.0, 99.5)
- added C3: 10uF, Capacitor_SMD:C_0603_1608Metric, F.Cu at (146.0, 95.5)
- U1: value ~ -> TPS542025DDCR
- moved C1 14.4 mm to (150.0, 99.5), turned to 180 degrees
- moved L1 14.4 mm to (150.3, 95.5)
- moved U1 0.86 mm to (141.5, 97.5)
Connections:
- C1 pad 2: +5V -> GND
- U1 pad 1: +5V -> GND
- U1 pad 4: unconnected-(U1-FB-Pad4) -> +5V
- U1 pad 6: unconnected-(U1-VBST-Pad6) -> Net-(U1-VBST)

Commit message: Changed component and updated docs
Parts:
- added C4: 47uF, Capacitor_SMD:C_1210_3225Metric, F.Cu at (141.5, 103.0)
- added C5: 47uF, Capacitor_SMD:C_1210_3225Metric, F.Cu at (136.0, 103.0)
- C1: value 22uF -> 47uF; footprint Capacitor_SMD:C_0603_1608Metric -> Capacitor_SMD:C_1210_3225Metric
- C2: value 1uF -> 0.1uF
- moved C1 14.2 mm to (136.0, 97.0), turned to 90 degrees
- moved L1 8.98 mm to (146.2, 103.5)
- moved U1 0.14 mm to (141.6, 97.5)
