File: pe/kicad-template/nile-dunning.kicad_sch (KiCad schematic)
At the start: 0 parts

Commit message: edmund let me in pops
Parts:
- added C1, C2, C3: C, Capacitor_SMD:C_0603_1608Metric, symbol Device:C
- added L1: L, inductor_footprint:IND_TAIYO_NRS4018_TAY, symbol Device:L
- added R1, R2: R, Resistor_SMD:R_0402_1005Metric, symbol Device:R
- added U2: TPS562202, Package_TO_SOT_SMD:SOT-563, symbol Regulator_Switching:TPS562202
Connections:
- new net: R1.1, R2.1, U2.6 (VFB)
- new net: C3.2, L1.1, U2.2 (SW)
- new net: C3.1, U2.4 (VBST)
- new net +12V: C1.1, U2.1 (VIN)
- new net +5V: C2.1, L1.2, R2.2
- new net GND: C1.2, C2.2, R1.2, U2.3 (GND)
- no-connect marks 0 -> 1
