File: pe/buck_converter/buck_converter.kicad_pcb (KiCad board)
At the start: 2 copper layers, 27.8 x 15.6 mm, 6 parts, among them Q1 BSS308PE

Commit message: Picked Parts, footprints
Parts:
- removed 5V_OUT1: ~, Connector_PinHeader_1.00mm:PinHeader_1x02_P1.00mm_Vertical_SMD_Pin1Left
- removed Q1: BSS308PE, Package_TO_SOT_SMD:SOT-23_Handsoldering
- added C2: 4.7uF, Capacitor_SMD:C_1206_3216Metric_Pad1.33x1.80mm_HandSolder, F.Cu at (57.0, 74.9)
- added C3: 0.01uF, Capacitor_SMD:C_0201_0603Metric_Pad0.64x0.40mm_HandSolder, F.Cu at (56.8, 69.9)
- added C4: 0.1uF, Capacitor_SMD:C_0201_0603Metric_Pad0.64x0.40mm_HandSolder, F.Cu at (66.1, 66.4)
- added C5: 0.01uF, Capacitor_SMD:C_0201_0603Metric_Pad0.64x0.40mm_HandSolder, F.Cu at (63.3, 75.1)
- added C6: 1000pF, Capacitor_SMD:C_0201_0603Metric_Pad0.64x0.40mm_HandSolder, F.Cu at (127.2, 87.5)
- added C7: 47pF, Capacitor_SMD:C_0201_0603Metric_Pad0.64x0.40mm_HandSolder, F.Cu at (127.2, 89.2)
- added C8: 47uF, Capacitor_SMD:C_1210_3225Metric_Pad1.33x2.70mm_HandSolder, F.Cu at (120.6, 65.0)
- added C9: 47uF, Capacitor_SMD:C_1210_3225Metric_Pad1.33x2.70mm_HandSolder, F.Cu at (120.6, 69.2)
- added R1: 332k, Resistor_SMD:R_0201_0603Metric_Pad0.64x0.40mm_HandSolder, F.Cu at (60.0, 69.9)
- added R2: 68.1k, Resistor_SMD:R_0201_0603Metric_Pad0.64x0.40mm_HandSolder, F.Cu at (60.0, 72.3)
- added R3: 29.4k, Resistor_SMD:R_0201_0603Metric_Pad0.64x0.40mm_HandSolder, F.Cu at (130.0, 84.0)
- added R4: 0, Resistor_SMD:R_0201_0603Metric_Pad0.64x0.40mm_HandSolder, F.Cu at (130.0, 85.7)
- added R5: 19.2k, Resistor_SMD:R_0201_0603Metric_Pad0.64x0.40mm_HandSolder, F.Cu at (130.0, 87.5)
- added R6: 3.25k, Resistor_SMD:R_0201_0603Metric_Pad0.64x0.40mm_HandSolder, F.Cu at (130.0, 89.2)
- added U1: TPS54331DR, Package_SO:SOIC-8_3.9x4.9mm_P1.27mm, F.Cu at (66.1, 71.6)
- C1: value C -> 4.7uF; footprint Capacitor_SMD:CP_Elec_10x10.5 -> Capacitor_SMD:C_1206_3216Metric_Pad1.33x1.80mm_HandSolder
- D1: value D -> B340A; footprint Diode_THT:D_DO-35_SOD27_P7.62mm_Horizontal -> Diode_SMD:D_SMA_Handsoldering
- L1: value L -> 6.8uH; footprint Inductor_SMD:L_0805_2012Metric -> Inductor_SMD:L_Bourns-SRN8040_8x8.15mm
- moved C1 64.5 mm to (53.1, 74.8), turned to -90 degrees
- moved 12V_IN1 56.5 mm to (48.1, 75.3), turned to 0 degrees
- moved D1 43.1 mm to (66.8, 83.0), turned to 180 degrees
- moved L1 29.1 mm to (81.7, 71.5)
Connections:
- 12V_IN1 pad 1: /12V_IN -> Net-(12V_IN1-Pin_1)
- C1 pad 1: Net-(5V_OUT1-Pin_1) -> Net-(12V_IN1-Pin_1)
- L1 pad 2: Net-(5V_OUT1-Pin_1) -> Net-(C8-Pad1)
Routing:
- net Net-(5V_OUT1-Pin_1): track 32.7 -> 0.00 mm
- net Net-(D1-K): track 8.23 -> 0.00 mm
- net /12V_IN: track 4.46 -> 0.00 mm
- removed copper zone on B.Cu, net /12V_IN
- removed copper zone on F.Cu, net GND
Other:
- board outline removed

Commit message: pcb layout complete
Parts:
- added 5V_OUT1: 12V_IN, Connector_PinHeader_2.54mm:PinHeader_1x02_P2.54mm_Vertical, F.Cu at (46.7, 65.5)
- 12V_IN1: footprint Connector_PinHeader_1.00mm:PinHeader_1x02_P1.00mm_Vertical_SMD_Pin1Left -> Connector_PinHeader_2.54mm:PinHeader_1x02_P2.54mm_Vertical
- moved R4 75.7 mm to (56.5, 67.7)
- moved R5 73.6 mm to (59.2, 67.7)
- moved R6 70.9 mm to (62.5, 67.8)
- moved R3 67.0 mm to (65.3, 66.6), turned to 90 degrees
- moved C6 62.8 mm to (68.1, 66.2), turned to -90 degrees
- moved C8 62.0 mm to (58.7, 62.1), turned to -90 degrees
- moved C7 60.9 mm to (70.9, 66.1), turned to -90 degrees
- moved C9 56.8 mm to (64.3, 62.2), turned to -90 degrees
- moved D1 23.4 mm to (53.4, 63.8), turned to -90 degrees
- moved L1 10.3 mm to (73.7, 78.1)
- moved C5 6.08 mm to (59.2, 79.6), turned to 180 degrees
- moved R2 5.16 mm to (57.7, 76.9), turned to 90 degrees
- moved C4 5.14 mm to (63.8, 71.0)
- moved R1 5.14 mm to (57.7, 74.4)
- moved C2 5.14 mm to (54.7, 79.5)
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Routing:
- net Net-(5V_OUT1-Pin_2): track 0.00 -> 52.4 mm
- net Net-(D1-K): track 0.00 -> 38.9 mm, vias 0 -> 5
- net Net-(12V_IN1-Pin_1): track 0.00 -> 24.8 mm
- net Net-(U1-VSENSE): track 0.00 -> 17.7 mm
- net Net-(U1-COMP): track 0.00 -> 15.8 mm
- net Net-(U1-EN): track 0.00 -> 5.34 mm
- net Net-(U1-BOOT): track 0.00 -> 4.15 mm
- net Net-(C6-Pad2): track 0.00 -> 3.03 mm
- net Net-(U1-SS): track 0.00 -> 2.59 mm
- net Net-(R4-Pad2): track 0.00 -> 1.87 mm
- added copper zone on F.Cu, net GND
Other:
- board outline added: 36.5 x 24.9 mm

Commit message: finishing touches
Parts:
- moved C5 1.96 mm to (61.0, 80.5)
Other:
- board size 36.5 x 24.9 mm -> 36.4 x 25.8 mm
Changed lines of the file:
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@@
 		(tags "resistor handsolder")
 		(property "Reference" "R3"
-			(at -0.0075 -1.2 90)
+			(at -1.5575 1.15 0)
 			(layer "F.SilkS")
 			(effects
@@
 		(tags "capacitor handsolder")
 		(property "Reference" "C6"
-			(at 1.9575 0.72 180)
+			(at -1.85 0.07 180)
 			(layer "F.SilkS")
 			(effects
@@
 		(tags "capacitor handsolder")
 		(property "Reference" "C7"
-			(at 0 -1.05 90)
+			(at 0.1 -1.45 90)
 			(layer "F.SilkS")
 			(effects
@@
 		(tags "capacitor handsolder")
 		(property "Reference" "C1"
-			(at 0 -1.85 90)
+			(at 3.5675 0.065 0)
 			(layer "F.SilkS")
 			(effects
@@
 		(tags "capacitor handsolder")
 		(property "Reference" "C2"
-			(at 0 -1.85 90)
+			(at 3.7275 0.005 0)
 			(layer "F.SilkS")
 			(effects
@@
 	(footprint "Capacitor_SMD:C_0201_0603Metric_Pad0.64x0.40mm_HandSolder"
 		(layer "F.Cu")
-		(at 59.1925 79.6 180)
+		(at 60.9575 80.45 180)
 		(descr "Capacitor SMD 0201 (0603 Metric), square (rectangular) end terminal, IPC-7351 nominal with elongated pad for handsoldering. (Body size source: https://www.vishay.com/docs/20052/crcw0201e3.pdf)")
 		(tags "capacitor handsolder")
 		(property "Reference" "C5"
-			(at 0.1075 -1.4 0)
+			(at 0.1075 -1.6 0)
 			(layer "F.SilkS")
 			(effects
@@
 		(tags "resistor handsolder")
 		(property "Reference" "R2"
-			(at 0 -1.05 90)
+			(at -2.3575 0 180)
 			(layer "F.SilkS")
 			(effects
@@
 	)
 	(gr_rect
-		(start 42.55 58.3)
-		(end 79 83.23)
+		(start 42.65 58.5)
+		(end 79.1 84.35)
 		(stroke
 			(width 0.0508)
@@
 		(start 49.3 65.485)
 		(end 49.3 65.8)
-		(width 0.508)
+		(width 0.254)
 		(layer "F.Cu")
 		(net "Net-(D1-K)")
@@
 		(start 70.7 78.3)
 		(end 70.9 78.1)
-		(width 0.508)
+		(width 0.254)
 		(layer "F.Cu")
 		(net "Net-(D1-K)")
@@
 		(start 53.445 61.34)
 		(end 49.3 65.485)
-		(width 0.508)
+		(width 0.254)
 		(layer "F.Cu")
 		(net "Net-(D1-K)")
@@
 		(start 68.4 78.3)
 		(end 70.7 78.3)
-		(width 0.508)
+		(width 0.254)
 		(layer "F.Cu")
 		(net "Net-(D1-K)")
@@
 		(start 49.3 65.8)
 		(end 54.5 71)
-		(width 0.508)
+		(width 0.254)
 		(layer "B.Cu")
 		(net "Net-(D1-K)")
@@
 		(start 68.4 78.3)
 		(end 68.4 73.9)
-		(width 0.508)
+		(width 0.254)
 		(layer "B.Cu")
 		(net "Net-(D1-K)")
@@
 		(start 68.4 73.9)
 		(end 67.275 72.775)
-		(width 0.508)
+		(width 0.254)
 		(layer "B.Cu")
 		(net "Net-(D1-K)")
@@
 		(start 67.275 72.775)
 		(end 65.5 71)
-		(width 0.508)
+		(width 0.254)
 		(layer "B.Cu")
 		(net "Net-(D1-K)")
@@
 		(start 54.5 71)
 		(end 65.5 71)
-		(width 0.508)
+		(width 0.254)
 		(layer "B.Cu")
 		(net "Net-(D1-K)")
@@
 	)
 	(segment
-		(start 47.35 69.8)
-		(end 54.0025 69.8)
+		(start 70.775 60.675)
+		(end 76.5 66.4)
 		(width 0.254)
 		(layer "F.Cu")
@@
 	)
 	(segment
-		(start 70.775 60.675)
-		(end 76.5 66.4)
+		(start 76.5 66.4)
+		(end 76.5 78.1)
 		(width 0.254)
 		(layer "F.Cu")
@@
 	)
 	(segment
-		(start 76.5 66.4)
-		(end 76.5 78.1)
+		(start 54.0025 69.8)
+		(end 56.1025 67.7)
+		(width 0.254)
+		(layer "F.Cu")
+		(net "Net-(5V_OUT1-Pin_2)")
+	)
+	(segment
+		(start 48.425 69.8)
+		(end 54.0025 69.8)
 		(width 0.254)
 		(layer "F.Cu")
@@
 		(start 56.092 61.508)
 		(end 56.092 67.7)
-		(width 0.508)
+		(width 0.254)
 		(layer "F.Cu")
 		(net "Net-(5V_OUT1-Pin_2)")
@@
 		(start 58.7 60.575)
 		(end 57.025 60.575)
-		(width 0.508)
+		(width 0.254)
 		(layer "F.Cu")
 		(net "Net-(5V_OUT1-Pin_2)")
 	)
 	(segment
-		(start 54.0025 69.8)
-		(end 56.1025 67.7)
+		(start 47.76 69.135)
+		(end 48.425 69.8)
 		(width 0.254)
 		(layer "F.Cu")
@@
 		(start 57.025 60.575)
 		(end 56.092 61.508)
-		(width 0.508)
+		(width 0.254)
 		(layer "F.Cu")
 		(net "Net-(5V_OUT1-Pin_2)")
@@
 		(start 59.95 68.05)
 		(end 59.6105 67.7105)
-		(width 0.508)
+		(width 0.254)
 		(layer "F.Cu")
 		(net "Net-(U1-VSENSE)")
@@
 		(start 66.262 70.262)
 		(end 64.762 68.762)
-		(width 0.508)
+		(width 0.254)
 		(layer "F.Cu")
 		(net "Net-(U1-VSENSE)")
@@
 		(start 62.280176 68.762)
 		(end 61.778 68.259824)
-		(width 0.508)
+		(width 0.254)
 		(layer "F.Cu")
 		(net "Net-(U1-VSENSE)")
@@
 		(start 59.6105 67.7105)
 		(end 59.6105 67.7)
-		(width 0.508)
+		(width 0.254)
 		(layer "F.Cu")
 		(net "Net-(U1-VSENSE)")
@@
 		(start 64.538 74.12229)
 		(end 66.262 72.39829)
-		(width 0.508)
+		(width 0.254)
 		(layer "F.Cu")
 		(net "Net-(U1-VSENSE)")
@@
 		(start 66.262 72.39829)
 		(end 66.262 70.262)
-		(width 0.508)
+		(width 0.254)
 		(layer "F.Cu")
 		(net "Net-(U1-VSENSE)")
@@
 		(start 64.762 68.762)
 		(end 62.280176 68.762)
-		(width 0.508)
+		(width 0.254)
 		(layer "F.Cu")
 		(net "Net-(U1-VSENSE)")
@@
 		(start 61.778 68.05)
 		(end 59.95 68.05)
-		(width 0.508)
+		(width 0.254)
 		(layer "F.Cu")
 		(net "Net-(U1-VSENSE)")
@@
 		(start 61.778 68.259824)
 		(end 61.778 68.05)
-		(width 0.508)
+		(width 0.254)
 		(layer "F.Cu")
 		(net "Net-(U1-VSENSE)")
@@
 		(start 64.538 77.342999)
 		(end 64.538 74.12229)
-		(width 0.508)
+		(width 0.254)
 		(layer "F.Cu")
 		(net "Net-(U1-VSENSE)")
@@
 		(start 66.275 78.105)
 		(end 65.300001 78.105)
-		(width 0.508)
+		(width 0.254)
 		(layer "F.Cu")
 		(net "Net-(U1-VSENSE)")
@@
 		(start 65.300001 78.105)
 		(end 64.538 77.342999)
-		(width 0.508)
+		(width 0.254)
 		(layer "F.Cu")
 		(net "Net-(U1-VSENSE)")
@@
 	)
 	(segment
-		(start 59.83 79.6)
-		(end 59.7375 79.6)
-		(width 0.254)
-		(layer "F.Cu")
-		(net "Net-(U1-SS)")
-	)
-	(segment
-		(start 60.01 79.3275)
-		(end 59.7375 79.6)
+		(start 61.325 78.105)
+		(end 61.5025 78.2825)
 		(width 0.254)
 		(layer "F.Cu")
@@
 	)
 	(segment
-		(start 61.325 78.105)
-		(end 59.83 79.6)
+		(start 61.5025 78.2825)
+		(end 61.5025 80.45)
 		(width 0.254)
 		(layer "F.Cu")
