File: LV-onboarding-kicad/LV-onboarding-kicad.kicad_sch (KiCad schematic)
At the start: 29 parts, among them J2 AiM Sports Pressure Sensors X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, J3 HASS 300, U1 ${SIM.PARAMS}, U10 74AHC1G04, U11 74AHC1G04, U12 74AHC1G04, U13 74AHC1G04, U2A ${SIM.PARAMS}, U2B ${SIM.PARAMS}, U3 ${SIM.PARAMS}, U4 74AHC1G08, U5 74AHC1G08, U6 74AHC1G08, U6A ${SIM.PARAMS}, U6B ${SIM.PARAMS}, U7 74AHC1G08, U8 74AHC1G08

Commit message: BSPD final work
removed page, conformed to standards, added rref for AiM sensor
Parts:
- R4: value FIND VALUE NEEEDED FOR THIS -> 26.5k
- R5: value FIND VALUE NEEDED -> 10k
Other:
- note removed: "where does the power for the sensors come from"
Changed lines of the file:
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@@
 		)
 	)
-	(text "where does the power for the sensors come from"
-		(exclude_from_sim no)
-		(at 224.282 112.268 0)
-		(effects
-			(font
-				(size 2.54 2.54)
-			)
-		)
-	)
 	(text "0.333v"
 		(exclude_from_sim no)
@@
 		)
 	)
-	(text "non inverting op amp"
-		(exclude_from_sim no)
-		(at 72.136 14.732 0)
-		(effects
-			(font
-				(size 1.27 1.27)
-			)
-		)
-	)
 	(text "0.333v"
 		(exclude_from_sim no)
@@
 	(text_box "creates 3.08V which is 46.3A from the battery\n(5kW trip)"
 		(exclude_from_sim no)
-		(at 23.5965 35.2414 0)
-		(size 21.3615 8.4466)
+		(at 23.3425 41.2258 0)
+		(size 21.3615 10.0822)
 		(margins 0.9525 0.9525 0.9525 0.9525)
 		(stroke
@@
 		(effects
 			(font
-				(size 0.508 0.508)
+				(size 1.27 1.27)
 			)
 		)
@@
 	)
 	(global_label "SENSORS_TRIPPED"
-		(shape input)
+		(shape output)
 		(at 180.34 93.98 0)
 		(fields_autoplaced yes)
@@
 			)
 		)
-		(property "Value" "FIND VALUE NEEDED"
+		(property "Value" "10k"
 			(at 27.94 134.6199 0)
 			(show_name no)
@@
 			)
 		)
-		(property "Value" "FIND VALUE NEEEDED FOR THIS"
+		(property "Value" "26.5k"
 			(at 27.94 124.4599 0)
 			(show_name no)
