File: LV-onboarding-kicad/sensorfault.kicad_sch (KiCad schematic)
At the start: 1 part, among them U9 74AHC1G02

Commit message: BSPD final work
removed page, conformed to standards, added rref for AiM sensor
Parts:
- removed U9: 74AHC1G02, Package_DFN_QFN:Nordic_AQFN-94-1EP_7x7mm_P0.4mm, symbol 74xGxx:74AHC1G02
Other:
- title: (none) -> Sample and Hold Circuit
