File: LV-onboarding-kicad/untitled.kicad_sch (KiCad schematic)
At the start: 9 parts, among them K1 Relay_SPST-NO, Q1 Q_NMOS_GDS, U14 LTC6994xS6-1, U16 74LVC2G02, U2 74LVC1G332

Commit message: BSPD final work
removed page, conformed to standards, added rref for AiM sensor
Parts:
- removed U2: 74LVC1G332, Package_TO_SOT_THT:TO-220-2_Vertical, symbol 74xGxx:74LVC1G332
- added U15: 74AHC1G02, symbol 74xGxx:74AHC1G02
- added U9: 74AHC1G02, Package_DFN_QFN:Nordic_AQFN-94-1EP_7x7mm_P0.4mm, symbol 74xGxx:74AHC1G02
Connections:
- net +5V: now also U15.5 (VCC), U9.5 (VCC)
- net GND: now also U15.3 (GND), U9.3 (GND)
- net SENSOR_FAULT: now also U15.2, U9.4
- net at U16.1: now also U15.4
- net at U14.6 (OUT): now also U15.1
- new net AiM_WORKING: U9.2
- new net HASS_WORKING: U9.1
Other:
- note removed: "check if the dual nor gate selection is good"
- note removed: "why sr latch instead of d flip flop"
- moved on the sheet: U16C
