File: lv/BMS PCB ONBOARDING.kicad_sch (KiCad schematic)
At the start: 142 parts, among them J3 512810598, J4 1053131202, J5 512810598, J6 1053131202, J701 430450200, J702 430450200, Q1 ZXTN25100DGTA, U1 BQ79616PAPRQ1

Commit message: UPDATE 5: Rail budget rework (TSREF -> CVDD) and footprint cleanup
Chip wiring:
- Move housekeeping pull-ups and quiet loads off TSREF onto CVDD,
  TSREF 30mA budget cannot cover the entire housekeeping rail
- Keep TSREF dedicated to its real job: NTC ratiometric bias
  for the temp-sense network only (switched off by default,
  tight load regulation, ~4mA intended load)
- CVDD is the always-on digital/IO LDO output from U1: it powers
  internal logic + IO supply and is the correct rail for external
  pull-ups, alerts, and light digital loads up to its rated limit
- Leave the 1uF bypass C205 and TP502 as the only TSREF loads
- All 16 VC rungs, 16 CB ladder rungs, and VC0-AVSS verified

Footprints fixed:
- R83 (100R VC15 sense): 2512 back to 0805 like the other 16
  sense resistors (R_0805_2012Metric_Pad1.20x1.40mm_HandSolder)
- FL701/FL702: KiCad:744242471 -> 744242471:744242471
- J4/J6 Nano-Fit: non-existent Nano-Fit_1054301102 ->
  Nanofit-1054301202-1x2SMD90Deg
- C701/C702/C707/C708: stripped " (1)" from library nickname
- Bundle all 143 custom .kicad_mod files into
  project_footprints.pretty inside the project and register
  every nickname in project + global fp-lib-table
  (KiCad only opens libraries whose folder ends in .pretty)
- All 142 netlist parts resolve: 0 missing footprints

Blocks on the sheet:
- Quit KiCad fully (Cmd+Q) so fp-lib-table and schematic
  reload from disk, then F8 Update PCB from Schematic
- Re-run ERC after the TSREF -> CVDD wire moves
- Confirm NEG5V charge-pump pin-type exclusion still holds

Pending:
- Place U1, 16-row VC/CB filter and balancing staircase,
  Q1 pre-regulator, and isolated comms blocks on PCB
- Route sense, balance, power, and differential comms traces
- Pour L2 solid AVSS ground plane and thermal copper for
  17x 10R 2512 balance resistors and Q1
- Run final DRC check

Learned:
- TSREF is a precision reference, not a supply rail,
  stacking housekeeping loads on it blows the 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
Parts:
- C701, C702, C707, C708: footprint 1206J2K00222KXR (1):CAPC3216X160N -> 1206J2K00222KXR:CAPC3216X160N
- FL701, FL702: footprint KiCad:744242471 -> 744242471:744242471
- J4, J6: footprint FS_4_Global_Footprint_Library:Nano-Fit_1054301102 -> FS_4_Global_Footprint_Library:Nanofit-1054301202-1x2SMD90Deg
- R83: footprint Resistor_SMD:R_2512_6332Metric -> Resistor_SMD:R_0805_2012Metric_Pad1.20x1.40mm_HandSolder
Connections:
- net CVDD: now also J3.5 (Pin_5), R12.1, R14.1, R5.1, R7.1, R8.1, R9.1
- net TSREF: no longer J3.5 (Pin_5), R12.1, R14.1, R5.1, R7.1, R8.1, R9.1

Commit message: UPDATE 7: board edge and mounting holes — connector half brought in as blocks
Board edge:
- The outline is on the board now, drawn as straight runs and rounded corners.
  Before this the file had no Edge.Cuts geometry at all, which is why DRC could
  not start and nothing could be plotted.
- The top-right corner is cut away: the area beyond the notch line is off the
  board, so the outline is not a plain rectangle.
- Every corner is an arc, and each mounting hole sits at the centre of one, so
  the corner relief is concentric with the fastener rather than cut beside it.
- Not closed yet: the right edge stops just short of where the next run picks
  it up, and a short segment lies on the left edge duplicating that part of it.
  Both leave free endpoints, which is what the outline check and every plot key
  off. The break is closed in the newer autosave; the duplicated segment is in
  all of them.

Mounting:
- The mounting holes are non-plated: a bare drill with no annular ring, and
  excluded from the BOM. At the tightest corners the ligament to the edge is
  thin but real; a washer up to the size the corner relief allows sits inside
  the arc, and anything wider overhangs it.
- Added on the sheet as well as the board - mounting-hole symbols with their
  own references - so schematic and board still agree after the board gained
  its footprints, and the used-designator list picked them up.

Blocks on the sheet:
- The connector / daisy-chain half came in from the far side of the sheet:
  a large share of the board moved and many parts also rotated between the
  first snapshot of the evening and the later save, most of them from
  beyond the right-hand end of the drawing area.
- The isolated block then moved as one piece: its parts - both daisy-chain
  connectors, the ladder resistors, the filter caps, the TVS pair and the
  chokes - shifted by a single rigid offset, with nothing inside the block
  changing relative to anything else in it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
Parts:
- added H1, H2, H3, H4: MountingHole, MountingHole:MountingHole_2.5mm, symbol Mechanical:MountingHole
