File: lv/ayush-maller.kicad_sch (KiCad schematic)
At the start: 6 parts, among them U1 INA333xxDGK

Commit message: updated bridge and INA333 instrumentation amplifier
Set gain from the expected 1% to 2% resistance change: R5 = 1.43 kΩ, so G ≈ 71 (G = 1 + 100 kΩ / R5).
Compression limit: G < 71.9 keeps the output above 0.05 V. At −2% the output is about 0.065 V, and at +2% it’s about 2.41 V.
Replaced the Ref ground connection with a REF3012 1.25 V reference  and a 0.1 µF capacitor
Made R2 a second gaugeat 90° to R1, which is mostly insensitive to thwstrain, so remeperature change is mostly accounted for
Parts:
- added C1: 100n, symbol Device:C
- added U2: REF3012, Package_TO_SOT_SMD:SOT-23, symbol Reference_Voltage:REF3012
- R2: value 350 -> GAUGE_90
- R5: value 200 -> 1.41k
Connections:
- net +3.3V: now also C1.1, U2.1 (IN)
- net GND: now also C1.2, U2.3 (GND); no longer U1.5 (Ref)
- new net VREF: U1.5 (Ref), U2.2 (OUT)
Other:
- moved on the sheet: R1, R2, R3, R4, R5, U1

Commit message: Assign footprints and update PCB from schematic
Parts:
- added C2: 100n, Capacitor_SMD:C_0603_1608Metric, symbol Device:C
- C1: footprint (none) -> Capacitor_SMD:C_0603_1608Metric
- R1, R2: footprint (none) -> Connector_PinHeader_2.54mm:PinHeader_1x02_P2.54mm_Vertical
- R3, R4: footprint (none) -> Resistor_SMD:R_0603_1608Metric
- R5: value 1.41k -> 2.49k; footprint (none) -> Resistor_SMD:R_0603_1608Metric
Connections:
- net +3.3V: now also C2.2
- net GND: now also C2.1
