File: pe/pe-onboarding-project/template/template.kicad_sch (KiCad schematic)
At the start: 15 parts, among them U2 TPS562208DDCR

Commit message: Add files via upload
Parts:
- removed C05: 0.1 µF, TPS562208DDCR:SOT95P280X110-6N, symbol Device:C
- added CO5: 0.1 µF, Capacitor_SMD:C_0603_1608Metric, symbol Device:C
- C1, C2, C3, C4: footprint Capacitor_SMD:C_0805_1608Metric -> Capacitor_SMD:C_0805_2012Metric
- C5: renamed from C6; footprint Capacitor_SMD:C_0805_1608Metric -> Capacitor_SMD:C_0805_2012Metric
- CBoot1, CO1, CO2, CO3, CO4: footprint TPS562208DDCR:SOT95P280X110-6N -> Capacitor_SMD:C_0603_1608Metric
- L1: footprint TPS562208DDCR:SOT95P280X110-6N -> FSCustom:IND_BOURNS_SRN6045
- R1: footprint Package_QFP:PQFP-160_28x28mm_P0.65mm -> Resistor_SMD:R_0603_1608Metric
- R2: footprint (none) -> Resistor_SMD:R_0603_1608Metric
- U2: footprint TPS562208DDCR:SOT95P280X110-6N -> FSCustom:DDC0006A_N
Connections:
- net GND: now also CO5.1; no longer C1.1, C2.1, C3.1, C4.1, C5.1, CO1.2, CO2.2, CO3.2, CO4.2, L1.1, R1.2, U2.3 (VIN)
- net at CBoot1.1, U2.2 (SW): now also L1.1; no longer L1.2
- new net VIN: C1.1, C2.1, C3.1, C4.1, C5.1, U2.3 (VIN)
- new net VOUT: CO1.2, CO2.2, CO3.2, CO4.2, CO5.2, L1.2, R1.2
Other:
- moved on the sheet: C1, C2, C3, C4, C5, CBoot1, CO1, CO2, CO3, CO4, L1, R1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
