File: pe/kicad-shunt/shunt.kicad_sch (KiCad schematic)
At the start: 0 parts

Commit message: Updated shunt schematics
Parts:
- added R1: R_Shunt 50µOhm, Package_SO:SOIC-8_3.9x4.9mm_P1.27mm, symbol Device:R_Shunt
- added R2: 210k, symbol Device:R_Small
- added R3: 90k, symbol Device:R_Small
- added U1: INA241A2-Q1, Package_SO:SOIC-8_3.9x4.9mm_P1.27mm, symbol Amplifier_Current:INA241A2xD
Connections:
- new net: R1.3, U1.1 (-)
- new net: R1.2, U1.8 (+)
- new net +5V: R2.1, U1.6 (V+)
- new net +BATT: R1.1
- new net 1.5_VREF2: R2.2, R3.1, U1.3 (REF2)
- new net GND: R3.2, U1.2 (GND), U1.4 (GND), U1.7 (REF1)
- new net V_Curr_Out: U1.5
Other:
- title: ${BOARD_TITLE} -> Current sense shunt

Commit message: Commiting the write up of my research Shunt_Research.pdf and the final version of the shunt schematic
Parts:
- removed R1: R_Shunt 50µOhm, Package_SO:SOIC-8_3.9x4.9mm_P1.27mm, symbol Device:R_Shunt
- added C1, C2: 0.1µF, formula_slug_footprint_library:128-TQFP-ECAP, symbol Device:C_Small
- added D12: PLZ3V3B-G3/H, Diode_SMD:D_SMF, symbol Device:D_Zener
- added U2: MCP6002-xMC, symbol Amplifier_Operational:MCP6004
- R2: value 210k -> 180k
- R3: value 90k -> 270k
- U1: value INA241A2-Q1 -> INA241A3-Q1
Connections:
- net +5V: now also C2.2, U2.4 (V+)
- net GND: now also C2.1, D12.2 (A), U2.11 (V-)
- net Vin-: now reaches U1.1 (-)
- net Vin+: now reaches U1.8 (+)
- net 1.5_VREF2: no longer names the net of R2.2, R3.1
- net 1.5_VREF2: now also U2.3 (+); no longer U1.3 (REF2)
- net V_Curr_Out renamed V_Out
- net V_Out: now also D12.1 (K)
- new net 3_VREF2: U1.3 (REF2), U2.1, U2.2 (-)
Other:
- note added: "GAIN = 50v/v"
- note added: "V_Out = 0 < V < 3"
- note added: "V_Out = Gain * (Vin+ - Vin-) + (Vref1 + Vref2)/2"
- moved on the sheet: R2, R3, U1
