File: pe/Charles Leong/template.kicad_sch (KiCad schematic)
At the start: 0 parts

Commit message: 10/16/26 12:24am kicad
Parts:
- added C1, C2, C3: 10μf, symbol Device:C
- added C4: 100nF, symbol Device:C
- added L1: L_Ferrite, symbol Device:L_Ferrite
- added U1: TPS54202DDC, Package_TO_SOT_SMD:SOT-23-6, symbol Regulator_Switching:TPS54202DDC
Connections:
- new net: C1.2, C2.2, C3.2, C4.2
- new net: L1.1, U1.6 (BOOT)
- new net Input: 10-15V: C1.1, C2.1, C3.1, C4.1, U1.3 (VIN)
Other:
- title: ${BOARD_TITLE} -> BUH_CONVERTER

Commit message: progress
12:49pm 10/16/2026
Parts:
- removed C1: 10μf, symbol Device:C
- added C5, C8: 100nF, symbol Device:C
- added C6, C7: 10μf, symbol Device:C
Connections:
- net GND: now reaches C2.2, C3.2, C4.2
- net GND: now also U1.1 (GND), U1.4 (FB), C6.2, C7.2, C8.2
- net at U1.2 (SW): now also L1.1, C5.2
- net at U1.6 (BOOT): now also C5.1; no longer L1.1
- net +5V: now reaches L1.2
- net +5V: now also C6.1, C7.1, C8.1
- net Input: 10-15V renamed +15V
- no-connect marks 0 -> 1
Other:
- moved on the sheet: C2, C3, C4, L1

Commit message: added descriptions
Parts:
- C2, C3, C6, C7: Digikey Part Number (none) -> 478-KGM55DR72A106MVDKR-ND; Digikey URL (none) -> https://www.digikey.com/en/products/detail/kyocera-avx/2220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; Manufacturer (none) -> KYOCERA AVX; Manufacturer Part Number (none) -> 22201C106MAT2A
- C4, C5, C8: Digikey Part Number (none) -> 399-C1210C104K5GACTUDKR-ND; Digikey URL (none) -> https://www.digikey.com/en/products/detail/kemet/C1210C104K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; Manufacturer (none) -> KEMET; Manufacturer Part Number (none) -> C1210C104K5GACTU
- L1: value L_Ferrite -> 12 µH; Digikey Part Number (none) -> 732-4529-6-ND; Digikey URL (none) -> https://www.digikey.com/en/products/detail/w%C3%BCrth-elekt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; Manufacturer (none) -> Würth Elektronik; Manufacturer Part Number (none) -> 744787120
Other:
- moved on the sheet: C2, C3, C4, C5, C6, C7, C8, L1, U1

Commit message: updated buck ic description
Parts:
- U1: value TPS54202DDC -> TPS542025DDCR; footprint Package_TO_SOT_SMD:SOT-23-6 -> (none); Digikey Part Number (none) -> 296-TPS542025DDCRDKR-ND; Digikey URL (none) -> https://www.digikey.com/en/products/detail/texas-instrument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; Manufacturer (none) -> Texas Instruments; Manufacturer Part Number (none) -> TPS542025DDCR
Changed lines of the file:
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@@
 			)
 		)
-		(property "Value" "TPS54202DDC"
+		(property "Value" "TPS542025DDCR"
 			(at 125.73 100.33 0)
 			(show_name no)
@@
 			)
 		)
-		(property "Footprint" "Package_TO_SOT_SMD:SOT-23-6"
+		(property "Footprint" ""
 			(at 127 116.84 0)
 			(hide yes)
@@
 			)
 		)
-		(property "Datasheet" "http://www.ti.com/lit/ds/symlink/tps54202.pdf"
+		(property "Datasheet" "https://www.ti.com/lit/ds/symlink/tps542025.pdf"
 			(at 118.11 99.06 0)
 			(hide yes)
@@
 			)
 		)
-		(property "Description" "2A, 4.5 to 28V Input, EMI Friendly integrated switch synchronous step-down regulator, pulse-skipping, SOT-23-6"
+		(property "Description" "Buck Switching Regulator IC Positive Fixed 5V 1 Output 2A SOT-23-6 Thin, TSOT-23-6"
 			(at 125.73 107.95 0)
 			(hide yes)
+			(show_name no)
+			(do_not_autoplace no)
+			(effects
+				(font
+					(size 1.27 1.27)
+				)
+			)
+		)
+		(property "Digikey Part Number" "296-TPS542025DDCRDKR-ND"
+			(at 125.73 107.95 0)
+			(hide yes)
+			(show_name no)
+			(do_not_autoplace no)
+			(effects
+				(font
+					(size 1.27 1.27)
+				)
+			)
+		)
+		(property "Digikey URL" "https://www.digikey.com/en/products/detail/texas-instruments/TPS542025DDCR/28738814"
+			(at 125.73 107.95 0)
+			(hide yes)
+			(show_name no)
+			(do_not_autoplace no)
+			(effects
+				(font
+					(size 1.27 1.27)
+				)
+			)
+		)
+		(property "Manufacturer" "Texas Instruments"
+			(at 125.73 107.95 0)
+			(hide yes)
+			(show_name no)
+			(do_not_autoplace no)
+			(effects
+				(font
+					(size 1.27 1.27)
+				)
+			)
+		)
+		(property "Manufacturer Part Number" "TPS542025DDCR"
+			(at 125.73 107.95 0)
+			(hide yes)
