File: pe/12V-buck/12V-buck.kicad_sch (KiCad schematic)
At the start: 9 parts, among them U1 TPS563208

Commit message: pcb update
Parts:
- removed R1: 100k, Resistor_SMD:R_0603_1608Metric_Pad0.98x0.95mm_HandSolder, symbol Device:R_US
- added J1: 12V, TerminalBlock_Phoenix:TerminalBlock_Phoenix_MKDS-1,5-2-5.08_1x02_P5.08mm_Horizontal, symbol Connector:Screw_Terminal_01x02
- added J2: 5V, TerminalBlock_Phoenix:TerminalBlock_Phoenix_MKDS-1,5-2-5.08_1x02_P5.08mm_Horizontal, symbol Connector:Screw_Terminal_01x02
- renumbered R2 to R1, R3 to R2
Connections:
- net +12V: now also U1.5 (EN), J1.1 (Pin_1)
- net +5V: now also J2.1 (Pin_1)
- net GND: now also J1.2 (Pin_2), J2.2 (Pin_2)
