File: lv/Amay-Singhania/Amay-Singhania.kicad_sch (KiCad schematic)
At the start: 24 parts

Commit message: lv and fw changes
Parts:
- removed R1, R10, R11, R12, R13, R15, R16, R17, R18, R19, R2, R3, R5: 350, Resistor_SMD:R_01005_0402Metric, symbol Device:R
- removed S1: StrainGaugeRef, StrainGauge:ReferenceStrainGauge, symbol Device:R_Variable
- removed S2, S3: StrainGaugeAxial, StrainGauge:Strain Gauge V1, symbol Device:R_Variable
- removed S5: StrainGaugeTorsion, StrainGauge:TorsionalGauge45deg, symbol Device:R_Variable
- added S7: StrainGaugeAxial, StrainGauge:Strain Gauge V1, symbol Device:R_Variable
- S6: value StrainGaugeTorsion -> StrainGaugeAxial; footprint StrainGauge:TorsionalGauge-45deg -> StrainGauge:Strain Gauge V1
Connections:
- net -IN Center Axial Gauge is gone; now on net GND: R14.2
- net +3V3: now also S7.2; no longer R14.1
- net +IN -45deg Torsion Gauge renamed Left Axial Gauge Unbuffered
- net +IN Center Axial Gauge renamed Center Axial Gauge Unbuffered
- net -IN Reference Gauge renamed 1V65 Unbuffered
- new net Right Axial Gauge Unbuffered: R14.1, S7.1
Other:
- moved on the sheet: R4, R8, R9, S4

Commit message: Final LV changes: updated research md file and finished schematic of strain gauges. Total BOM: 9.61!
Parts:
- added C15, C16, C17: 100nF, Package_TO_SOT_SMD:TSOT-23-5, symbol Device:C
- added C18: 0.1uF, Package_TO_SOT_SMD:TSOT-23-5, symbol Device:C
- added C19, C20, C21, C22, C23, C24: C, Package_TO_SOT_SMD:TSOT-23-5, symbol Device:C
- added IC1: TLV4888DR, SOIC127P600X175-14N, symbol TLV4888DR:TLV4888DR
- added JP2, JP3, JP4, JP5, JP6: (no value), Package_TO_SOT_SMD:SOT-23-6_Handsoldering, symbol formula_slug_symbol_library:SolderJumper_Open_Small
- added R1, R10, R11, R2, R3: R, Package_DIP:DIP-8_W7.62mm, symbol Device:R
- added R5: 350, Resistor_SMD:R_01005_0402Metric, symbol Device:R
- added S5: StrainGaugeReference, StrainGauge:ReferenceStrainGauge, symbol Device:R_Variable
- added SW5: SW_DIP_x04, symbol Switch:SW_DIP_x04
- added SW6: SW_DIP_x02, symbol Switch:SW_DIP_x02
- added U5: ADS122C14IRTER, RTE0016C-IPC_A, symbol ADS122C14:ADS122C14IRTER
Connections:
- net +3V3: now also C15.1, C16.1, S5.2, SW5.6, SW6.3, U5.13 (DVDD), U5.15 (AVDD)
- net Center Axial Gauge Unbuffered: now also IC1.5 (+IN_B)
- net GND: now also C15.2, C16.2, C17.1, C18.2, C19.1, C19.2, C20.1, C21.1, C22.1, C23.1, C24.1, IC1.11 (V-), R5.2, SW5.5, SW6.4, U5.14 (GND), U5.17 (Thermal_Pad)
- net Left Axial Gauge Unbuffered: now also IC1.12 (+IN_D)
- net Right Axial Gauge Unbuffered: now also IC1.10 (+IN_C)
- net 1V65 Unbuffered renamed 1V65
- net 1V65: now also JP6.2, U5.8 (AIN7_GPIO3_DRDY_CLKIN_N)
- new net: JP5.2, JP6.1, U5.2 (AIN1), U5.4 (AIN3), U5.6 (AIN5_REFN_GPIO1)
- new net: IC1.1 (OUT_A), IC1.2 (-IN_A), R1.2, R11.2
- new net: IC1.13 (-IN_D), IC1.14 (OUT_D), JP4.2, R10.1
- new net: IC1.6 (-IN_B), IC1.7 (OUT_B), JP2.2, R2.1
- new net: IC1.8 (OUT_C), IC1.9 (-IN_C), JP3.2, R3.1
- new net: SW6.1, SW6.2, U5.10 (A1)
- new net: C17.2, U5.16 (REFOUT)
- new net: SW5.1, SW5.2, SW5.3, SW5.4, U5.9 (A0)
- new net +5V: C18.1, IC1.4 (V+)
- new net ADC SCL: SW5.7, U5.12 (SCL)
- new net ADC SDA: SW5.8, U5.11 (SDA)
- new net Center Axial Gauge: C20.2, JP2.1, R2.2, U5.3 (AIN2)
- new net Left Axial Gauge: C22.2, JP4.1, R10.2, U5.1 (AIN0)
- new net Reference Gauge Unbuffered: IC1.3 (+IN_A), R5.1, S5.1
- new net Right Axial Gauge: C21.2, JP3.1, R3.2, U5.5 (AIN4_REFP_GPIO0)
- new net SG Reference: C23.2, R1.1, U5.7 (AIN6_GPIO2_FAULT_N)
- new net SG Reference Filtered: C24.2, JP5.1, R11.1
Other:
- note added: "128x Gain set in firmware"
- note added: "Select I2C Address Using Dip Switches"
- note added: "Tau = 1/f(sample)"

Commit message: small changes
Other:
- note added: "$1.620/IC"
- note added: "$7.489/IC"
Changed lines of the file:
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@@
+		)
+	)
+	(text "$7.489/IC"
+		(exclude_from_sim no)
+		(at 227.838 66.294 0)
+		(effects
+			(font
+				(size 1.27 1.27)
+			)
 		)
 	)
@@
 		(effects
 			(font
+				(size 1.27 1.27)
+			)
+		)
+	)
+	(text "$1.620/IC"
+		(exclude_from_sim no)
+		(at 92.456 166.116 0)
+		(effects
+			(font
