File: pe/zander-hong/zander-hong.kicad_sch (KiCad schematic)
At the start: 8 parts, among them U1 AP62300TWU

Commit message: updated schematic to add doc link
Other:
- note added: "PE Onboarding DOC"
Changed lines of the file:
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@@
 		(comment 3 "${COMMENT2}")
+	)
+	(text "PE Onboarding DOC"
+		(exclude_from_sim no)
+		(at 128.016 136.398 0)
+		(effects
+			(font
+				(size 1.27 1.27)
+			)
+			(href "https://docs.google.com/document/d/13sFLwHUCCrR32Jd7PrSwRqvHXB84yX7d5dig93GgXCQ/edit?usp=sharing")
+		)
 	)
 	(text "C1: Input Filtering Cap\nC2 & C2A: Output Filtering Cap in parallel to account for DC Bias Derating\nC3: Bootstrap Cap to power gate for N channel MOSFET"
