File: lv/gavin-barron/gavin-barron.kicad_sch (KiCad schematic)
At the start: 0 parts

Commit message: Complete BSPD schematic: power, brake input, current input, and logic sheets.
Parts:
- added J101: Brake_IN, symbol Connector_Generic:Conn_01x02
- added J102: Power_IN, symbol Connector_Generic:Conn_01x02
- added J103: Current_IN, symbol Connector_Generic:Conn_01x03
- added J104: BSPD_OUT, symbol Connector_Generic:Conn_01x02
Connections:
- new net +12V: J102.1 (Pin_1)
- new net Brake_Input/BRAKE_SIG: J101.1 (Pin_1)
- new net Current_Input/HASS_OUT: J103.1 (Pin_1)
- new net Current_Input/HASS_REF: J103.2 (Pin_2)
- new net GND: J101.2 (Pin_2), J102.2 (Pin_2), J103.3 (Pin_3), J104.2 (Pin_2)
- new net Logic/BSPD_OK: J104.1 (Pin_1)
Other:
- added sheet Brake_Input (brake_input.kicad_sch)
- added sheet Current_Input (current_input.kicad_sch)
- added sheet Logic (logic.kicad_sch)
- added sheet Power (power.kicad_sch)
