File: pe/charles-leong-buhconverter-kicad/charlesleong.kicad_sch (KiCad schematic)
At the start: 9 parts, among them U1 TPS542025DDCR

Commit message: stuff
Parts:
- U1: footprint (none) -> Package_TO_SOT_SMD:SOT-23-6
Other:
- title: BUH_CONVERTER -> $[BUH_CONVERTER]
Changed lines of the file:
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@@
 	(paper "A")
 	(title_block
-		(title "BUH_CONVERTER")
+		(title "$[BUH_CONVERTER]")
 		(date "${CURRENT_DATE}")
 		(rev "${REVISION}")
@@
 		)
 		(instances
-			(project "template"
+			(project "charlesleong"
 				(path "/e994741c-7c7d-4124-9d00-43b883baa61d"
 					(reference "#PWR04")
@@
 		)
 		(instances
-			(project "template"
+			(project "charlesleong"
 				(path "/e994741c-7c7d-4124-9d00-43b883baa61d"
 					(reference "C6")
@@
 		)
 		(instances
-			(project "template"
+			(project "charlesleong"
 				(path "/e994741c-7c7d-4124-9d00-43b883baa61d"
 					(reference "C5")
@@
 		)
 		(instances
-			(project "template"
+			(project "charlesleong"
 				(path "/e994741c-7c7d-4124-9d00-43b883baa61d"
 					(reference "C4")
@@
 		)
 		(instances
-			(project "template"
+			(project "charlesleong"
 				(path "/e994741c-7c7d-4124-9d00-43b883baa61d"
 					(reference "C3")
@@
 		)
 		(instances
-			(project "template"
+			(project "charlesleong"
 				(path "/e994741c-7c7d-4124-9d00-43b883baa61d"
 					(reference "#PWR05")
@@
 		)
 		(instances
-			(project "template"
+			(project "charlesleong"
 				(path "/e994741c-7c7d-4124-9d00-43b883baa61d"
 					(reference "#FLG01")
@@
 		)
 		(instances
-			(project "template"
+			(project "charlesleong"
 				(path "/e994741c-7c7d-4124-9d00-43b883baa61d"
 					(reference "#PWR01")
@@
 		)
 		(instances
-			(project "template"
+			(project "charlesleong"
 				(path "/e994741c-7c7d-4124-9d00-43b883baa61d"
 					(reference "C2")
@@
 		)
 		(instances
-			(project "template"
+			(project "charlesleong"
 				(path "/e994741c-7c7d-4124-9d00-43b883baa61d"
 					(reference "#FLG02")
@@
 		)
 		(instances
-			(project "template"
+			(project "charlesleong"
 				(path "/e994741c-7c7d-4124-9d00-43b883baa61d"
 					(reference "#FLG03")
@@
 		)
 		(instances
-			(project "template"
+			(project "charlesleong"
 				(path "/e994741c-7c7d-4124-9d00-43b883baa61d"
 					(reference "C8")
@@
 			)
 		)
-		(property "Footprint" ""
+		(property "Footprint" "Package_TO_SOT_SMD:SOT-23-6"
 			(at 127 116.84 0)
 			(hide yes)
@@
 		)
 		(instances
-			(project "template"
+			(project "charlesleong"
 				(path "/e994741c-7c7d-4124-9d00-43b883baa61d"
 					(reference "U1")
@@
 		)
 		(instances
-			(project "template"
+			(project "charlesleong"
 				(path "/e994741c-7c7d-4124-9d00-43b883baa61d"
 					(reference "L1")
@@
 		)
 		(instances
-			(project "template"
+			(project "charlesleong"
 				(path "/e994741c-7c7d-4124-9d00-43b883baa61d"
 					(reference "C7")

Commit message: added pcb footprints
Parts:
- C2, C3, C6, C7: footprint (none) -> Capacitor_SMD:C_2220_5750Metric_Pad1.97x5.40mm_HandSolder
- C4, C5, C8: footprint (none) -> Capacitor_SMD:C_1210_3225Metric_Pad1.33x2.70mm_HandSolder
- L1: footprint (none) -> formula_slug_footprint_library:L_Wurth_WE-PD2SR-7850
Changed lines of the file:
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@@
 			)
 		)
-		(property "Footprint" ""
+		(property "Footprint" "Capacitor_SMD:C_2220_5750Metric_Pad1.97x5.40mm_HandSolder"
 			(at 162.2552 115.57 0)
 			(hide yes)
@@
 			)
 		)
-		(property "Footprint" ""
+		(property "Footprint" "Capacitor_SMD:C_1210_3225Metric_Pad1.33x2.70mm_HandSolder"
 			(at 140.6652 107.95 0)
 			(hide yes)
@@
 			)
 		)
-		(property "Footprint" ""
+		(property "Footprint" "Capacitor_SMD:C_1210_3225Metric_Pad1.33x2.70mm_HandSolder"
 			(at 105.1052 113.03 0)
 			(hide yes)
@@
 			)
 		)
-		(property "Footprint" ""
+		(property "Footprint" "Capacitor_SMD:C_2220_5750Metric_Pad1.97x5.40mm_HandSolder"
 			(at 93.6752 113.03 0)
 			(hide yes)
@@
 			)
 		)
-		(property "Footprint" ""
+		(property "Footprint" "Capacitor_SMD:C_2220_5750Metric_Pad1.97x5.40mm_HandSolder"
 			(at 82.2452 113.03 0)
 			(hide yes)
@@
 			)
 		)
-		(property "Footprint" ""
+		(property "Footprint" "Capacitor_SMD:C_1210_3225Metric_Pad1.33x2.70mm_HandSolder"
 			(at 187.6552 115.57 0)
 			(hide yes)
@@
 			)
 		)
-		(property "Footprint" ""
+		(property "Footprint" "formula_slug_footprint_library:L_Wurth_WE-PD2SR-7850"
 			(at 154.94 107.95 0)
 			(hide yes)
@@
 			)
 		)
-		(property "Footprint" ""
+		(property "Footprint" "Capacitor_SMD:C_2220_5750Metric_Pad1.97x5.40mm_HandSolder"
 			(at 174.9552 115.57 0)
 			(hide yes)

Commit message: pcb components
Parts:
- renumbered C2 to C1, C3 to C2, C4 to C3, C5 to C4, C6 to C5, C7 to C6, C8 to C7
Changed lines of the file:
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@@
 		(dnp no)
 		(fields_autoplaced yes)
-		(property "Reference" "C6"
+		(property "Reference" "C5"
 			(at 165.1 110.4899 0)
 			(show_name no)
@@
 			(project "charlesleong"
 				(path "/e994741c-7c7d-4124-9d00-43b883baa61d"
-					(reference "C6")
+					(reference "C5")
 					(unit 1)
 				)
@@
 		(dnp no)
 		(fields_autoplaced yes)
-		(property "Reference" "C5"
+		(property "Reference" "C4"
 			(at 143.51 102.8699 0)
 			(show_name no)
@@
 			(project "charlesleong"
 				(path "/e994741c-7c7d-4124-9d00-43b883baa61d"
-					(reference "C5")
+					(reference "C4")
 					(unit 1)
 				)
@@
 		(dnp no)
 		(fields_autoplaced yes)
-		(property "Reference" "C4"
+		(property "Reference" "C3"
 			(at 107.95 107.9499 0)
 			(show_name no)
@@
 			(project "charlesleong"
 				(path "/e994741c-7c7d-4124-9d00-43b883baa61d"
-					(reference "C4")
+					(reference "C3")
 					(unit 1)
 				)
@@
 		(dnp no)
 		(fields_autoplaced yes)
-		(property "Reference" "C3"
+		(property "Reference" "C2"
 			(at 96.52 107.9499 0)
 			(show_name no)
@@
 			(project "charlesleong"
 				(path "/e994741c-7c7d-4124-9d00-43b883baa61d"
-					(reference "C3")
+					(reference "C2")
 					(unit 1)
 				)
@@
 		(dnp no)
 		(fields_autoplaced yes)
-		(property "Reference" "C2"
+		(property "Reference" "C1"
 			(at 85.09 107.9499 0)
 			(show_name no)
@@
 			(project "charlesleong"
 				(path "/e994741c-7c7d-4124-9d00-43b883baa61d"
-					(reference "C2")
+					(reference "C1")
 					(unit 1)
 				)
@@
 		(dnp no)
 		(fields_autoplaced yes)
-		(property "Reference" "C8"
+		(property "Reference" "C7"
 			(at 190.5 110.4899 0)
 			(show_name no)
@@
 			(project "charlesleong"
 				(path "/e994741c-7c7d-4124-9d00-43b883baa61d"
-					(reference "C8")
+					(reference "C7")
 					(unit 1)
 				)
@@
 		(dnp no)
 		(fields_autoplaced yes)
-		(property "Reference" "C7"
+		(property "Reference" "C6"
 			(at 177.8 110.4899 0)
 			(show_name no)
@@
 			(project "charlesleong"
 				(path "/e994741c-7c7d-4124-9d00-43b883baa61d"
-					(reference "C7")
+					(reference "C6")
 					(unit 1)
 				)
