File: lv/riddhi-mundhra/bspd_circuit/bspd_circuit.kicad_sch (KiCad schematic)
At the start: 8 parts, among them U1 OPA196xDGK, U2 OPA196xDGK, U3 TLV172IDCK

Commit message: update circuit
Connections:
- net GND: no longer R1.1
Changed lines of the file:
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@@
 	(wire
 		(pts
-			(xy 87.63 118.11) (xy 83.82 118.11)
+			(xy 104.14 113.03) (xy 104.14 114.3)
 		)
 		(stroke
@@
 	(wire
 		(pts
-			(xy 104.14 113.03) (xy 104.14 114.3)
+			(xy 116.84 74.93) (xy 118.11 74.93)
 		)
 		(stroke
@@
 	(wire
 		(pts
-			(xy 116.84 74.93) (xy 118.11 74.93)
+			(xy 95.25 123.19) (xy 99.06 123.19)
 		)
 		(stroke
@@
 	(wire
 		(pts
-			(xy 95.25 123.19) (xy 99.06 123.19)
+			(xy 130.81 72.39) (xy 132.08 73.66)
 		)
 		(stroke
@@
 		)
 	)
-	(wire
-		(pts
-			(xy 130.81 72.39) (xy 132.08 73.66)
-		)
-		(stroke
-			(width 0)
-			(type default)
-		)
-	)
 	(symbol
 		(lib_id "Amplifier_Operational:TLV172IDCK")
@@
 					(unit 1)
 				)
-			)
-		)
-	)
-	(symbol
-		(lib_id "power:GND")
-		(at 83.82 118.11 270)
-		(unit 1)
-		(body_style 1)
-		(exclude_from_sim no)
-		(in_bom yes)
-		(on_board yes)
-		(in_pos_files yes)
-		(dnp no)
-		(fields_autoplaced yes)
-		(property "Reference" "#PWR05"
-			(at 77.47 118.11 0)
-			(hide yes)
-			(show_name no)
-			(do_not_autoplace no)
-			(effects
-				(font
-					(size 1.27 1.27)
-				)
-			)
-		)
-		(property "Value" "GND"
-			(at 78.74 118.11 0)
-			(show_name no)
-			(do_not_autoplace no)
-			(effects
-				(font
-					(size 1.27 1.27)
-				)
-			)
-		)
-		(property "Footprint" ""
-			(at 83.82 118.11 0)
-			(hide yes)
-			(show_name no)
-			(do_not_autoplace no)
-			(effects
-				(font
-					(size 1.27 1.27)
-				)
-			)
-		)
-		(property "Datasheet" ""
-			(at 83.82 118.11 0)
-			(hide yes)
-			(show_name no)
-			(do_not_autoplace no)
-			(effects
-				(font
-					(size 1.27 1.27)
-				)
-			)
-		)
-		(property "Description" "Power symbol creates a global label with name \"GND\" , ground"
-			(at 83.82 118.11 0)
-			(hide yes)
-			(show_name no)
-			(do_not_autoplace no)
-			(effects
-				(font
-					(size 1.27 1.27)
-				)
-			)
-		)
-		(pin "1"
-		)
-		(instances
-			(project "bspd_circuit"
-				(path "/384d8ed3-10e0-45cc-a390-f82c2bfa0c8b"
-					(reference "#PWR05")
-					(unit 1)
-				)
