File: lv/lorenzo-serrano/op-amp-comparator-v1.kicad_sch (KiCad schematic)
At the start: 3 parts, among them U1 LM358

Commit message: Added low-pass filter and screw-pot
Parts:
- removed R2: 10k, symbol Device:R
- added C1: 1u, symbol Device:C
- added R2: 100k, symbol Device:R_Trim
- added R3: 8.2k, symbol Device:R
Connections:
- net GND: now also C1.2, R2.2
- net Vref: now also R2.1
- net +5V renamed 5V
- new net V_filtered: C1.1, R3.2
Other:
- note added: "V_filtered (0.5V - 4.5V)"
- note removed: "Vbrk (0.5V - 4.5V)"
