File: pe/maheer-grang/maheer-grang.kicad_pcb (KiCad board)
At the start: 2 copper layers, 25 x 19.5 mm, 11 parts, among them U1 AP62300TWU

Commit message: final draft for pe onboarding
Parts:
- added C0: 10 µF, Capacitor_SMD:C_0603_1608Metric_Pad1.08x0.95mm_HandSolder, F.Cu at (140.5, 93.9)
- C1, C2: footprint Capacitor_SMD:C_1206_3216Metric -> Capacitor_SMD:C_0603_1608Metric_Pad1.08x0.95mm_HandSolder
- L1: value B82464P4472M000 -> 4.7 µH; footprint Inductor_SMD:L_10.4x10.4_H4.8 -> Inductor_SMD:L_Pulse_PA4332
- moved C5 16.1 mm to (139.0, 83.8)
- moved C4 16.0 mm to (139.0, 82.2)
- moved L1 12.0 mm to (143.0, 84.0), turned to 90 degrees
- moved C1 2.57 mm to (139.0, 93.9)
- moved C2 1.62 mm to (137.5, 93.9)
- moved C3 1.00 mm to (139.0, 85.5)
- moved R1 0.50 mm to (143.0, 87.5)
- moved R2 0.50 mm to (143.0, 89.0)
- moved R3 0.50 mm to (138.6, 90.5)
- moved R4 0.50 mm to (142.0, 90.5)
Routing:
- net Net-(C4-Pad1): track 33.2 -> 15.4 mm
- net Net-(U1-SW): track 6.92 -> 9.15 mm
- net Net-(U1-IN): track 7.39 -> 9.26 mm
- net Net-(U1-FB): track 4.04 -> 2.76 mm
- net Net-(U1-BST): track 2.72 -> 1.72 mm
- net Net-(U1-EN): track 5.92 -> 5.42 mm
- net GNDREF: track 10.5 -> 10.9 mm, vias 7 -> 8
Other:
- board size 25 x 19.5 mm -> 10.5 x 16.5 mm
