File: pe/maheer-grang/maheer-grang.kicad_sch (KiCad schematic)
At the start: 11 parts, among them U1 AP62300TWU

Commit message: final draft for pe onboarding
Parts:
- added C0: 10 µF, Capacitor_SMD:C_0603_1608Metric_Pad1.08x0.95mm_HandSolder, symbol Device:C_Small
- C1, C2: footprint Capacitor_SMD:C_1206_3216Metric -> Capacitor_SMD:C_0603_1608Metric_Pad1.08x0.95mm_HandSolder; Digikey Part Number 490-6518-1-ND -> 490-12737-1-ND; Digikey URL https://www.digikey.com/en/products/detail/murata-electronics/GRM31CR71E106KA12L/2345330 -> https://www.digikey.com/en/products/detail/murata-electronics/GRM188R61E106MA73J/4905347; Manufacturer Part Number GRM31CR71E106KA12L -> GRM188R61E106MA73J
- L1: value B82464P4472M000 -> 4.7 µH; footprint Inductor_SMD:L_10.4x10.4_H4.8 -> Inductor_SMD:L_Pulse_PA4332; Digikey Part Number 495-77086-1-ND -> 4044-CSEG0430H-4R7MTR-ND; Digikey URL (none) -> https://www.digikey.com/en/products/detail/codaca/CSEG0430H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; Manufacturer TDK -> CODACA; Manufacturer Part Number B82464P4472M000 -> CSEG0430H-4R7M
Connections:
- net GNDREF: now also C0.2
- net at C1.1, C2.1, R3.1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: now also C0.1
