File: pe/buck-convertor-project/buck_convertor/buck_convertor.kicad_sch (KiCad schematic)
At the start: 0 parts

Commit message: components placed, wiring started
Parts:
- added C1: 10uF, Package_QFP:PQFP-160_28x28mm_P0.65mm, symbol Device:C
- added C2, C3: 0.1uF, symbol Device:C
- added C4, C5: 22uF, symbol Device:C
- added C6: 75pF, symbol Device:C
- added J1: 12V INPUT, Connector_Audio:Jack_XLR_Neutrik_NC3FAAH_Horizontal, symbol Connector_Generic:Conn_01x02
- added J2: 5V OUTPUT, Connector_Audio:Jack_XLR_Neutrik_NC3FAAH_Horizontal, symbol Connector_Generic:Conn_01x02
- added L1: 15uH, Package_QFP:PQFP-160_28x28mm_P0.65mm, symbol Device:L
- added R1: 100k, symbol Device:R
- added R2: 13.3k, symbol Device:R
- added R3: 510k, symbol Device:R
- added R4: 105k, symbol Device:R
- added U1: TPS54202DDC, Package_TO_SOT_SMD:SOT-23-6, symbol Regulator_Switching:TPS54202DDC
Connections:
- new net: C1.1, C2.1, J1.1 (Pin_1), U1.3 (VIN)

Commit message: buck converter schematic finished
Connections:
- net at C3.1: now also U1.6 (BOOT)
- net at C3.2: now also L1.1, U1.2 (SW)
- net at J2.1 (Pin_1): now also C4.1, C5.1, L1.2
- net GND: now reaches J2.2 (Pin_2)
- net GND: now also C1.2, C2.2, C4.2, C5.2, J1.2 (Pin_2), R2.2, R4.2, U1.1 (GND)
- net FB: now reaches U1.4 (FB)
- net EN: now reaches R3.2
- net EN: now also R4.1
- net at R2.1: now also C6.2, R1.2
- net at R1.1: now also C6.1
Other:
- moved on the sheet: C2, C3, C4, C5, C6, J2, L1, R1, R2, R3, R4

Commit message: fixed text labels, disconnected electrical labels in schematic
Connections:
- net FB: now also C6.2, R1.2, R2.1
- net VIN: now also C1.1, C2.1, J1.1 (Pin_1), R3.1, U1.3 (VIN)
- net VOUT: now also C4.1, C5.1, C6.1, J2.1 (Pin_1), L1.2, R1.1
Other:
- note added: "ENABLE DIVIDER"
- note added: "FEEDBACK DIVIDER"
Changed lines of the file:
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@@
 		(comment 3 "${COMMENT2}")
 	)
+	(text "ENABLE DIVIDER\n"
+		(exclude_from_sim no)
+		(at 108.966 124.714 0)
+		(effects
+			(font
+				(size 1.27 1.27)
+			)
+		)
+	)
+	(text "FEEDBACK DIVIDER\n"
+		(exclude_from_sim no)
+		(at 164.846 125.73 0)
+		(effects
+			(font
+				(size 1.27 1.27)
+			)
+		)
+	)
 	(junction
 		(at 156.21 130.81)
@@
 	)
 	(junction
+		(at 196.85 105.41)
+		(diameter 0)
+		(color 0 0 0 0)
+	)
+	(junction
 		(at 118.11 139.7)
 		(diameter 0)
@@
 	(wire
 		(pts
+			(xy 205.74 101.6) (xy 196.85 105.41)
+		)
+		(stroke
+			(width 0)
+			(type default)
+		)
+	)
+	(wire
+		(pts
 			(xy 92.71 95.25) (xy 88.9 95.25)
 		)
@@
 	(wire
 		(pts
-			(xy 194.31 105.41) (xy 203.2 105.41)
-		)
-		(stroke
-			(width 0)
-			(type default)
-		)
-	)
-	(wire
-		(pts
 			(xy 118.11 149.86) (xy 118.11 153.67)
 		)
@@
 	(wire
 		(pts
-			(xy 182.88 105.41) (xy 194.31 105.41)
+			(xy 182.88 105.41) (xy 203.2 105.41)
 		)
 		(stroke
@@
 	)
 	(label "VOUT"
-		(at 157.48 129.54 0)
+		(at 156.21 129.54 0)
 		(effects
 			(font
@@
 	)
 	(label "EN"
-		(at 125.73 139.7 0)
+		(at 127 139.7 0)
 		(effects
 			(font
@@
 	)
 	(label "FB"
-		(at 162.56 143.51 0)
+		(at 167.64 144.78 0)
 		(effects
 			(font
@@
 	)
 	(label "VIN"
-		(at 119.38 128.27 0)
-		(effects
-			(font
-				(size 1.27 1.27)
-			)
-			(justify left bottom)
-		)
-	)
-	(label "FEEDBACK DIVIDER"
-		(at 142.24 125.73 0)
+		(at 118.11 127 0)
 		(effects
 			(font
@@
 	)
 	(label "VIN"
-		(at 106.68 91.44 0)
+		(at 106.68 92.71 0)
 		(effects
 			(font
@@
 	)
 	(label "VOUT"
-		(at 190.5 104.14 0)
-		(effects
-			(font
-				(size 1.27 1.27)
-			)
-			(justify left bottom)
-		)
-	)
-	(label "ENABLE DIVIDER"
-		(at 102.87 125.73 0)
+		(at 205.74 101.6 0)
 		(effects
 			(font
@@
 	)
 	(label "EN"
-		(at 125.73 104.14 0)
-		(effects
-			(font
+		(at 127 105.41 0)
+		(effects
+			(font
