File: pe/matthew-riffle/matthew-riffle.kicad_sch (KiCad schematic)
At the start: 11 parts, among them U1 TPP302080-T6TR

Commit message: updated schematic with revised capacitor selection
Parts:
- C5, C6: Digikey Part Number 4713-GMC10X5R226M10NTCT-ND -> 490-13243-1-ND; Digikey URL https://www.digikey.com/en/products/detail/cal-chip-electro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 -> https://www.digikey.com/en/products/detail/murata-electroni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; Manufacturer Cal-Chip Electronics, Inc. -> Murata Electronics; Manufacturer Part Number GMC10X5R226M10NT -> GRM187R61A226ME15D
Changed lines of the file:
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@@
 			)
 		)
-		(property "Datasheet" "https://www.susumu.co.jp/english/product/rg.html"
+		(property "Datasheet" "https://www.susumu.co.jp/dl/?filename=n_catalog_partition01_en.pdf&type=application%2Fpdf"
 			(at 167.64 105.41 0)
 			(hide yes)
@@
 			)
 		)
-		(property "Datasheet" "https://www.murata.com/en-us/products/productdetail?partno=GRM188R61E106MA73%23"
+		(property "Datasheet" "https://search.murata.co.jp/Ceramy/image/img/A01X/G101/ENG/GRM188R61E106MA73-01A.pdf"
 			(at 83.82 90.17 0)
 			(hide yes)
@@
 			)
 		)
-		(property "Description" "Unpolarized capacitor"
+		(property "Description" "Ceramic capacitor"
 			(at 83.82 90.17 0)
 			(hide yes)
@@
 			)
 		)
-		(property "Datasheet" "https://calchip.com/wp-content/uploads/2025/05/GMC-Series-3.pdf"
+		(property "Datasheet" "https://mm.digikey.com/Volume0/opasdata/d220001/medias/docus/8942/490_Chip_Multilayer_CAT2021_MLCC.pdf"
 			(at 200.66 87.63 0)
 			(hide yes)
@@
 			)
 		)
-		(property "Description" "Unpolarized capacitor"
+		(property "Description" "Ceramic capacitor"
 			(at 200.66 87.63 0)
 			(hide yes)
@@
 			)
 		)
-		(property "Digikey Part Number" "4713-GMC10X5R226M10NTCT-ND"
+		(property "Digikey Part Number" "490-13243-1-ND"
 			(at 200.66 87.63 0)
 			(hide yes)
@@
 			)
 		)
-		(property "Digikey URL" "https://www.digikey.com/en/products/detail/cal-chip-electronics-inc/GMC10X5R226M10NT/22461275"
+		(property "Digikey URL" "https://www.digikey.com/en/products/detail/murata-electronics/GRM187R61A226ME15D/5877406"
 			(at 200.66 87.63 0)
 			(hide yes)
@@
 			)
 		)
-		(property "Manufacturer Part Number" "GMC10X5R226M10NT"
+		(property "Manufacturer Part Number" "GRM187R61A226ME15D"
 			(at 200.66 87.63 0)
 			(hide yes)
@@
 			)
 		)
-		(property "Manufacturer" "Cal-Chip Electronics, Inc."
+		(property "Manufacturer" "Murata Electronics"
 			(at 200.66 87.63 0)
 			(hide yes)
@@
 			)
 		)
-		(property "Description" "Unpolarized capacitor"
+		(property "Description" "Ceramic capacitor"
 			(at 100.33 90.17 0)
 			(hide yes)
@@
 			)
 		)
-		(property "Datasheet" "https://www.murata.com/en-us/products/productdetail?partno=GRM188R61E106MA73%23"
+		(property "Datasheet" "https://search.murata.co.jp/Ceramy/image/img/A01X/G101/ENG/GRM188R61E106MA73-01A.pdf"
 			(at 67.31 90.17 0)
 			(hide yes)
@@
 			)
 		)
-		(property "Description" "Unpolarized capacitor"
+		(property "Description" "Ceramic capacitor"
 			(at 67.31 90.17 0)
 			(hide yes)
@@
 			)
 		)
-		(property "Datasheet" "https://www.susumu.co.jp/english/product/rg.html"
+		(property "Datasheet" "https://www.susumu.co.jp/dl/?filename=n_catalog_partition01_en.pdf&type=application%2Fpdf"
 			(at 167.64 87.63 0)
 			(hide yes)
@@
 			)
 		)
-		(property "Datasheet" "https://calchip.com/wp-content/uploads/2025/05/GMC-Series-3.pdf"
+		(property "Datasheet" "https://mm.digikey.com/Volume0/opasdata/d220001/medias/docus/8942/490_Chip_Multilayer_CAT2021_MLCC.pdf"
 			(at 184.15 87.63 0)
 			(hide yes)
@@
 			)
 		)
-		(property "Description" "Unpolarized capacitor"
+		(property "Description" "Ceramic capacitor"
 			(at 184.15 87.63 0)
 			(hide yes)
@@
 			)
 		)
-		(property "Digikey Part Number" "4713-GMC10X5R226M10NTCT-ND"
+		(property "Digikey Part Number" "490-13243-1-ND"
 			(at 184.15 87.63 0)
 			(hide yes)
@@
 			)
 		)
-		(property "Digikey URL" "https://www.digikey.com/en/products/detail/cal-chip-electronics-inc/GMC10X5R226M10NT/22461275"
+		(property "Digikey URL" "https://www.digikey.com/en/products/detail/murata-electronics/GRM187R61A226ME15D/5877406"
 			(at 184.15 87.63 0)
 			(hide yes)
@@
 			)
 		)
-		(property "Manufacturer Part Number" "GMC10X5R226M10NT"
+		(property "Manufacturer Part Number" "GRM187R61A226ME15D"
 			(at 184.15 87.63 0)
 			(hide yes)
@@
 			)
 		)
-		(property "Manufacturer" "Cal-Chip Electronics, Inc."
+		(property "Manufacturer" "Murata Electronics"
 			(at 184.15 87.63 0)
 			(hide yes)

Commit message: added PCB layout and onboarding documentation
Parts:
- added J1: INPUT, Connector_Wire:SolderWire-0.75sqmm_1x02_P4.8mm_D1.25mm_OD2.3mm, symbol Connector_Generic:Conn_01x02
- added J2: OUTPUT, Connector_Wire:SolderWire-0.75sqmm_1x02_P4.8mm_D1.25mm_OD2.3mm, symbol Connector_Generic:Conn_01x02
Connections:
- net +12V: now also J1.1 (Pin_1)
- net +5V: now also J2.1 (Pin_1)
- net GND: now also J1.2 (Pin_2), J2.2 (Pin_2)
Changed lines of the file:
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@@
 		)
 	)
+(symbol (lib_id "Connector_Generic:Conn_01x02") (at 76.2 144.78 0) (unit 1)
+      (exclude_from_sim no) (in_bom no) (on_board yes) (dnp no)
+      (property "Reference" "J1" (at 76.2 139.7 0)  (effects (font (size 1.27 1.27)))) (property "Value" "INPUT" (at 76.2 152.4 0)  (effects (font (size 1.27 1.27)))) (property "Footprint" "Connector_Wire:SolderWire-0.75sqmm_1x02_P4.8mm_D1.25mm_OD2.3mm" (at 76.2 144.78 0) (hide yes) (effects (font (size 1.27 1.27)))) (property "Datasheet" "" (at 76.2 144.78 0) (hide yes) (effects (font (size 1.27 1.27)))) (property "Description" "PCB solder wire pads: pin 1 +12V, pin 2 GND; no separate connector component" (at 76.2 144.78 0) (hide yes) (effects (font (size 1.27 1.27))))
+      (pin "1") (pin "2")
+      (instances (project "matthew-riffle" (path "/cf8f5d00-2a5e-5240-b793-3a4da5fda1d7" (reference "J1") (unit 1)))))
+(wire (pts (xy 63.5 144.78) (xy 71.12 144.78)) (stroke (width 0) (type default)))
+(label "+12V" (at 63.5 144.78 0) (effects (font (size 1.27 1.27)) (justify left bottom)))
+(wire (pts (xy 63.5 147.32) (xy 71.12 147.32)) (stroke (width 0) (type default)))
+(label "GND" (at 63.5 147.32 0) (effects (font (size 1.27 1.27)) (justify left bottom)))
+(symbol (lib_id "Connector_Generic:Conn_01x02") (at 182.88 144.78 0) (unit 1)
+      (exclude_from_sim no) (in_bom no) (on_board yes) (dnp no)
+      (property "Reference" "J2" (at 182.88 139.7 0)  (effects (font (size 1.27 1.27)))) (property "Value" "OUTPUT" (at 182.88 152.4 0)  (effects (font (size 1.27 1.27)))) (property "Footprint" "Connector_Wire:SolderWire-0.75sqmm_1x02_P4.8mm_D1.25mm_OD2.3mm" (at 182.88 144.78 0) (hide yes) (effects (font (size 1.27 1.27)))) (property "Datasheet" "" (at 182.88 144.78 0) (hide yes) (effects (font (size 1.27 1.27)))) (property "Description" "PCB solder wire pads: pin 1 +5V, pin 2 GND; no separate connector component" (at 182.88 144.78 0) (hide yes) (effects (font (size 1.27 1.27))))
+      (pin "1") (pin "2")
+      (instances (project "matthew-riffle" (path "/cf8f5d00-2a5e-5240-b793-3a4da5fda1d7" (reference "J2") (unit 1)))))
+(wire (pts (xy 170.18 144.78) (xy 177.8 144.78)) (stroke (width 0) (type default)))
+(label "+5V" (at 170.18 144.78 0) (effects (font (size 1.27 1.27)) (justify left bottom)))
+(wire (pts (xy 170.18 147.32) (xy 177.8 147.32)) (stroke (width 0) (type default)))
+(label "GND" (at 170.18 147.32 0) (effects (font (size 1.27 1.27)) (justify left bottom)))
 )
