File: pe/connor-hassfeld/connor-hassfeld.kicad_sch (KiCad schematic)
At the start: 0 parts

Commit message: Add 12V input connector and input capacitors (J1, C1, C2)
Parts:
- added C1: 10uF, Capacitor_SMD:C_1206_3216Metric_Pad1.33x1.80mm_HandSolder, symbol Device:C
- added C2: 100nF, Capacitor_SMD:C_0603_1608Metric_Pad1.08x0.95mm_HandSolder, symbol Device:C
- added J1: Conn_01x02, Connector_PinHeader_2.54mm:PinHeader_1x02_P2.54mm_Vertical, symbol Connector_Generic:Conn_01x02
Connections:
- new net +12V: C1.1, C2.1, J1.1 (Pin_1)
- new net GND: C1.2, C2.2, J1.2 (Pin_2)
Other:
- note added: "GLV: [10, 15]"

Commit message: Add notes on input capacitor roles and personalize J1 value
Parts:
- J1: value Conn_01x02 -> Connor_01x02
Other:
- note added: "c1 (bulk capacitor)"
- note added: "c2 = high f capacitor (next to chip)"
Changed lines of the file:
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@@
 		(comment 3 "${COMMENT2}")
+	)
+	(text ""
+		(exclude_from_sim no)
+		(at 22.86 81.026 0)
+		(effects
+			(font
+				(size 1.27 1.27)
+			)
+		)
+	)
+	(text "c1 (bulk capacitor)"
+		(exclude_from_sim no)
+		(at 22.606 79.248 0)
+		(effects
+			(font
+				(size 1.27 1.27)
+			)
+		)
 	)
 	(text "GLV: [10, 15]"
@@
 			)
 			(justify left bottom)
+		)
+	)
+	(text "c2 = high f capacitor (next to chip)"
+		(exclude_from_sim no)
+		(at 31.242 82.55 0)
+		(effects
+			(font
+				(size 1.27 1.27)
+			)
 		)
 	)
@@
 		)
 		(instances
-			(project ""
+			(project "connor-hassfeld"
 				(path "/e994741c-7c7d-4124-9d00-43b883baa61d"
 					(reference "#PWR03")
@@
 		)
 		(instances
-			(project ""
+			(project "connor-hassfeld"
 				(path "/e994741c-7c7d-4124-9d00-43b883baa61d"
 					(reference "C2")
@@
 		)
 		(instances
-			(project ""
+			(project "connor-hassfeld"
 				(path "/e994741c-7c7d-4124-9d00-43b883baa61d"
 					(reference "#PWR02")
@@
 			)
 		)
-		(property "Value" "Conn_01x02"
+		(property "Value" "Connor_01x02"
 			(at 27.94 106.68 0)
 			(show_name no)
@@
 		)
 		(instances
-			(project ""
+			(project "connor-hassfeld"
 				(path "/e994741c-7c7d-4124-9d00-43b883baa61d"
 					(reference "J1")
@@
 		)
 		(instances
-			(project ""
+			(project "connor-hassfeld"
 				(path "/e994741c-7c7d-4124-9d00-43b883baa61d"
 					(reference "#PWR04")
@@
 		)
 		(instances
-			(project ""
+			(project "connor-hassfeld"
 				(path "/e994741c-7c7d-4124-9d00-43b883baa61d"
 					(reference "C1")
@@
 		)
 		(instances
-			(project ""
+			(project "connor-hassfeld"
 				(path "/e994741c-7c7d-4124-9d00-43b883baa61d"
 					(reference "#PWR01")

Commit message: Add TPS54202 buck regulator and boot capacitor (U1, C3)
Parts:
- added C3: 100nF, Capacitor_SMD:C_0603_1608Metric_Pad1.08x0.95mm_HandSolder, symbol Device:C
- added U1: Our Buck IC Chip TPS54202DDCR, Package_TO_SOT_SMD:TSOT-23-6_HandSoldering, symbol Regulator_Switching:TPS54202DDC
Connections:
- net +12V: now also U1.3 (VIN)
- net GND: now also U1.1 (GND)
- new net: C3.2, U1.2 (SW)
- new net Conn for bootcaps: C3.1, U1.6 (BOOT)
- no-connect marks 0 -> 1

Commit message: Add 10uH output inductor and switch node (L1)
Parts:
- added L1(inductorrrr): SRP6540-100M, Inductor_SMD:L_Coilcraft_XAL6060-XXX, symbol Device:L
Connections:
- net SW: now reaches C3.2, U1.2 (SW)
- net SW: now also L1(inductorrrr).1
- new net +5V: L1(inductorrrr).2

Commit message: Add output capacitors and 5V output connector (C4-C7, J2)
Also update L1 to the Bourns SRP6540-100M: footprint, datasheet,
part numbers, and a project-local footprint from the datasheet's
recommended land pattern.
Parts:
- added C4, C5, C6: 22uF, Capacitor_SMD:C_0805_2012Metric_Pad1.18x1.45mm_HandSolder, symbol Device:C
- added C7: 100nF, Capacitor_SMD:C_0603_1608Metric_Pad1.08x0.95mm_HandSolder, symbol Device:C
- added J2: Connor_01x02, Connector_PinHeader_2.54mm:PinHeader_1x02_P2.54mm_Vertical, symbol Connector_Generic:Conn_01x02
- L1(inductorrrr): footprint Inductor_SMD:L_Coilcraft_XAL6060-XXX -> connor-hassfeld:L_Bourns_SRP6540; Digi PN 2457-XGL6060-153MEC-ND -> SRP6540-100MCT-ND; Digi URL https://www.digikey.com/en/products/detail/coilcraft/XGL606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 -> https://www.digikey.com/en/products/detail/bourns-inc/SRP65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; MFG Coilcraft -> Bourns Inc.; MFG PN XGL6060-153MEC -> SRP6540-100M
Connections:
- net +5V: now also C4.1, C5.1, C6.1, C7.1, J2.1 (Pin_1)
- net GND: now also C4.2, C5.2, C6.2, C7.2, J2.2 (Pin_2)
Other:
- note added: "+5V w 2A"
- note added: "all the samsung CL21A226MOQNNNE"
- note added: "output version of c2"

Commit message: Add feedback divider and feed-forward capacitor (R1, R2, C8)
Parts:
- added C8: 68pF, Capacitor_SMD:C_0603_1608Metric_Pad1.08x0.95mm_HandSolder, symbol Device:C
- added R1: 100k, Resistor_SMD:R_0603_1608Metric_Pad0.98x0.95mm_HandSolder, symbol Device:R
- added R2: 13.3k, Resistor_SMD:R_0603_1608Metric_Pad0.98x0.95mm_HandSolder, symbol Device:R
Connections:
- net +5V: now also C8.1, R1.1
- net GND: now also R2.2
- net FB: now reaches U1.4 (FB)
- net FB: now also C8.2, R1.2, R2.1
Other:
- note added: "Feed forward capacitor across R1"
- note added: "Voltage divider from output to FB pin (voltage transition)"

Commit message: Add design and layout notes, power flags included
Also update U1's symbol from the KiCad library (clears the last ERC warning).
Other:
- note added: "1. C1/C2 right at VIN-GND pins; C2 (100nF) closest"
- note added: "2. Keep SW copper (U1.2 - C3 - L1) small and short"
- note added: "3. C3 boot cap tight between BOOT and SW"
- note added: "4. FB trace away from SW/L1; R1 top taps the output caps"
- note added: "5. GND pour top+bottom, vias around U1"
- note added: "6. +12V/+5V/GND traces >= 30 mil"
- note added: "CONNOR J. HASSFELD'S 12V -> 5V / 2A BUCK CONVERTER (TI TPS54202, 500 kHz fixed)"
- note added: "EN: I left floating to enable, NEVER tie EN to 12 V (it will merk the converter)"
- note added: "ERC power flags: tell KiCad these nets are driven (+12V and GND from J1, +5V from the converter)"
- note added: "Inductor: 10 mew h, 2.33A, Isat -> 4A"
- note added: "Layout notes for making the PCB"
- note added: "More details than whats listed below can be found in activity 2 of the 'Connor Hassfeld - Power Elecronics Onboarding' doc"
- note added: "Output Voltage: V_out = 0.596 x (1+R_1/R_2) = 5.08 V"
- note added: "Specs: 10-15V in, 5V / 2A out, 500kHz"

Commit message: Fill in title block and fix L1 reference designator
Parts:
- renumbered L1(inductorrrr) to L1
Changed lines of the file:
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@@
 		(in_pos_files yes)
 		(dnp no)
-		(property "Reference" "L1(inductorrrr)"
-			(at 133.096 99.314 90)
+		(property "Reference" "L1"
+			(at 127.508 99.568 90)
 			(show_name no)
 			(do_not_autoplace no)
@@
 			(project "connor-hassfeld"
 				(path "/e994741c-7c7d-4124-9d00-43b883baa61d"
-					(reference "L1(inductorrrr)")
+					(reference "L1")
 					(unit 1)
 				)
