File: arush-kadam/arush-kadam.kicad_pcb (KiCad board)
At the start: 2 copper layers, 0 parts

Commit message: Added documentation PDF and fixed capacitor names on schematic
Parts:
- added C1: 10uF, Capacitor_SMD:C_0805_2012Metric, F.Cu at (1.73, 1.00)
- added C10: 22uF, Capacitor_SMD:C_0805_2012Metric, F.Cu at (6.17, 4.01)
- added C11: 22uF, Capacitor_SMD:C_0805_2012Metric, F.Cu at (6.17, 7.03)
- added C12: 22uF, Capacitor_SMD:C_0805_2012Metric, F.Cu at (6.17, 10.0)
- added C13: 22uF, Capacitor_SMD:C_0805_2012Metric, F.Cu at (6.17, 13.0)
- added C2: 10uF, Capacitor_SMD:C_0805_2012Metric, F.Cu at (1.73, 4.01)
- added C3: 10uF, Capacitor_SMD:C_0805_2012Metric, F.Cu at (1.73, 7.03)
- added C4: 10uF, Capacitor_SMD:C_0805_2012Metric, F.Cu at (1.73, 10.0)
- added C7: 22uF, Capacitor_SMD:C_0805_2012Metric, F.Cu at (1.73, 13.0)
- added C8: 22uF, Capacitor_SMD:C_0805_2012Metric, F.Cu at (1.73, 16.1)
- added C9: 22uF, Capacitor_SMD:C_0805_2012Metric, F.Cu at (6.17, 1.00)
- added R1: 158kΩ, Resistor_SMD:R_0603_1608Metric_Pad0.98x0.95mm_HandSolder, F.Cu at (10.6, 0.76)
- added R2: 30.1kΩ, Resistor_SMD:R_0603_1608Metric_Pad0.98x0.95mm_HandSolder, F.Cu at (10.6, 3.27)
