File: pe/dr-schematic/dr.kicad_sch (KiCad schematic)
At the start: 0 parts

Commit message: Buck converter components added to KiCad schematic and lined up, values defined.
Parts:
- added C1, C2: 22u, symbol Device:C
- added C3: 4.7u, symbol Device:C
- added C4, C5: 100n, symbol Device:C
- added L1: 10uH, symbol Device:L
- added R1: 100k, symbol Device:R
- added R2: 13.7k, symbol Device:R
- added U1: LMR51420XFDDCR, Package_TO_SOT_SMD:SOT-23-6, symbol Regulator_Switching:TPS54202DDC
Connections:
- new net: C5.2, L1.1, U1.2 (SW)
- new net: C5.1, U1.6 (BOOT)
- new net +12V: C3.1, C4.1, U1.3 (VIN)
- new net GND: C3.2, C4.2
Other:
- title: ${BOARD_TITLE} -> ${Schematic - Onboarding Buck Converter}
