File: pe/je-buck-converter/je-buck-converter.kicad_sch (KiCad schematic)
At the start: 6 parts, among them Q1 PMOS

Commit message: minor schematic + simulation adjustments
Parts:
- removed C1: 3uF, symbol Device:C
- renumbered C2 to C1
Other:
- moved on the sheet: V1
Changed lines of the file:
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@@
-	)
-	(junction
-		(at 109.22 99.06)
-		(diameter 0)
-		(color 0 0 0 0)
 	)
 	(junction
@@
 	)
 	(junction
-		(at 109.22 81.28)
+		(at 127 81.28)
 		(diameter 0)
 		(color 0 0 0 0)
 	)
 	(junction
-		(at 127 81.28)
+		(at 109.22 96.52)
 		(diameter 0)
 		(color 0 0 0 0)
@@
 	(wire
 		(pts
-			(xy 109.22 93.98) (xy 109.22 99.06)
+			(xy 109.22 93.98) (xy 109.22 96.52)
 		)
 		(stroke
@@
 	(wire
 		(pts
-			(xy 92.71 81.28) (xy 92.71 85.09)
-		)
-		(stroke
-			(width 0)
-			(type default)
-		)
-	)
-	(wire
-		(pts
-			(xy 92.71 99.06) (xy 109.22 99.06)
+			(xy 109.22 81.28) (xy 109.22 86.36)
 		)
 		(stroke
@@
 	(wire
 		(pts
-			(xy 92.71 95.25) (xy 92.71 99.06)
-		)
-		(stroke
-			(width 0)
-			(type default)
-		)
-	)
-	(wire
-		(pts
 			(xy 132.08 81.28) (xy 127 81.28)
 		)
@@
 	(wire
 		(pts
+			(xy 109.22 96.52) (xy 109.22 99.06)
+		)
+		(stroke
+			(width 0)
+			(type default)
+		)
+	)
+	(wire
+		(pts
 			(xy 109.22 81.28) (xy 113.03 81.28)
 		)
@@
 	(wire
 		(pts
-			(xy 92.71 81.28) (xy 109.22 81.28)
-		)
-		(stroke
-			(width 0)
-			(type default)
-		)
-	)
-	(wire
-		(pts
-			(xy 109.22 81.28) (xy 109.22 86.36)
-		)
-		(stroke
-			(width 0)
-			(type default)
-		)
-	)
-	(wire
-		(pts
 			(xy 109.22 99.06) (xy 127 99.06)
 		)
@@
 			(width 0)
 			(type default)
-		)
-	)
-	(symbol
-		(lib_id "Device:C")
-		(at 109.22 90.17 0)
-		(unit 1)
-		(body_style 1)
-		(exclude_from_sim no)
-		(in_bom yes)
-		(on_board yes)
-		(in_pos_files yes)
-		(dnp no)
-		(fields_autoplaced yes)
-		(property "Reference" "C1"
-			(at 113.03 88.8999 0)
-			(show_name no)
-			(do_not_autoplace no)
-			(effects
-				(font
-					(size 1.27 1.27)
-				)
-				(justify left)
-			)
-		)
-		(property "Value" "3uF"
-			(at 113.03 91.4399 0)
-			(show_name no)
-			(do_not_autoplace no)
-			(effects
-				(font
-					(size 1.27 1.27)
-				)
-				(justify left)
-			)
-		)
-		(property "Footprint" ""
-			(at 110.1852 93.98 0)
-			(hide yes)
-			(show_name no)
-			(do_not_autoplace no)
-			(effects
-				(font
-					(size 1.27 1.27)
-				)
-			)
-		)
-		(property "Datasheet" ""
-			(at 109.22 90.17 0)
-			(hide yes)
-			(show_name no)
-			(do_not_autoplace no)
-			(effects
-				(font
-					(size 1.27 1.27)
-				)
-			)
-		)
-		(property "Description" "Unpolarized capacitor"
-			(at 109.22 90.17 0)
-			(hide yes)
-			(show_name no)
-			(do_not_autoplace no)
-			(effects
-				(font
-					(size 1.27 1.27)
-				)
-			)
-		)
-		(pin "2"
-		)
-		(pin "1"
-		)
-		(instances
-			(project "je-buck-converter"
-				(path "/e994741c-7c7d-4124-9d00-43b883baa61d"
-					(reference "C1")
-					(unit 1)
-				)
-			)
 		)
 	)
@@
 		(dnp no)
 		(fields_autoplaced yes)
-		(property "Reference" "C2"
+		(property "Reference" "C1"
 			(at 148.59 88.8999 0)
 			(show_name no)
@@
 			(project "je-buck-converter"
 				(path "/e994741c-7c7d-4124-9d00-43b883baa61d"
-					(reference "C2")
+					(reference "C1")
 					(unit 1)
 				)
@@
 	(symbol
 		(lib_id "Simulation_SPICE:VDC")
-		(at 92.71 90.17 0)
+		(at 109.22 91.44 0)
 		(unit 1)
 		(body_style 1)
@@
 		(fields_autoplaced yes)
 		(property "Reference" "V1"
-			(at 96.52 88.7701 0)
+			(at 113.03 90.0401 0)
 			(show_name no)
 			(do_not_autoplace no)
@@
 		)
 		(property "Value" "12V"
-			(at 96.52 91.3101 0)
+			(at 113.03 92.5801 0)
 			(show_name no)
 			(do_not_autoplace no)
@@
 		)
 		(property "Footprint" ""
-			(at 92.71 90.17 0)
+			(at 109.22 91.44 0)
 			(hide yes)
 			(show_name no)
@@
 		)
 		(property "Datasheet" "https://ngspice.sourceforge.io/docs/ngspice-html-manual/manual.xhtml#sec_Independent_Sources_for"
-			(at 92.71 90.17 0)
+			(at 109.22 91.44 0)
 			(hide yes)
 			(show_name no)
@@
 		)
 		(property "Description" "Voltage source, DC"
-			(at 92.71 90.17 0)
+			(at 109.22 91.44 0)
 			(hide yes)
 			(show_name no)
@@
 		)
 		(property "Sim.Pins" "1=+ 2=-"
-			(at 92.71 90.17 0)
+			(at 109.22 91.44 0)
 			(hide yes)
 			(show_name no)
@@
 		)
 		(property "Sim.Type" "DC"
-			(at 92.71 90.17 0)
+			(at 109.22 91.44 0)
 			(hide yes)
 			(show_name no)
@@
 		)
 		(property "Sim.Device" "V"
-			(at 92.71 90.17 0)
+			(at 109.22 91.44 0)
 			(hide yes)
 			(show_name no)
@@
 		)
 		(property "Digikey Part Number" ""
-			(at 92.71 90.17 0)
+			(at 109.22 91.44 0)
 			(hide yes)
 			(show_name no)
@@
 		)
 		(property "Digikey URL" ""
-			(at 92.71 90.17 0)
+			(at 109.22 91.44 0)
 			(hide yes)
 			(show_name no)
@@
 		)
 		(property "Manufacturer" ""
-			(at 92.71 90.17 0)
+			(at 109.22 91.44 0)
 			(hide yes)
 			(show_name no)
@@
 		)
 		(property "Manufacturer Part Number" ""
-			(at 92.71 90.17 0)
-			(hide yes)
-			(show_name no)
+			(at 109.22 91.44 0)
+			(hide yes)
+			(show_name no)

Commit message: atrocious pcb
Parts:
- removed D1: D_Schottky, symbol Device:D_Schottky
- removed Q1: PMOS, symbol Simulation_SPICE:PMOS
- removed V1: 12V, symbol Simulation_SPICE:VDC
- added C2: 13n, Capacitor_SMD:C_0201_0603Metric, symbol Device:C
- added CR1: MBRS360T3G, MBRS360T3G:DIODE_SMC_7P15X6P25_ONS-M, symbol MBRS360T3G:MBRS360T3G
- added J1, J2: Conn_01x02_Pin, Connector_PinSocket_2.54mm:PinSocket_1x02_P2.54mm_Vertical, symbol Connector:Conn_01x02_Pin
- added R1: 33k, Resistor_SMD:R_0603_1608Metric, symbol Device:R_US
- added U1: TPS5405DR, TPS5405DR:SOIC127P599X175-8N, symbol TPS5405DR:TPS5405DR
- C1: value 3uF -> 2.2uF; footprint (none) -> Capacitor_SMD:C_0201_0603Metric
- L1: value 10uH -> 7uH; footprint (none) -> Inductor_SMD:L_Bourns-SRU1028_10.0x10.0mm; Manufacturer Part Number (none) -> PF0560.702NL
Connections:
- net at C1.1, L1.2: now also J2.2 (Pin_2), U1.5 (VSENSE)
- net GND: now reaches C1.2
- net GND: now also C2.2, CR1.1, J1.2 (Pin_2), J2.1 (Pin_1), R1.2, U1.7 (GND)
- net at L1.1: now also CR1.2, U1.8 (LX)
- new net: J1.1 (Pin_1), U1.2 (VIN)
- new net: C2.1, U1.4 (SS)
- new net: R1.1, U1.3 (ROSC)
Other:
- note added: "V_in = 12V"
- note added: "V_out ~ 5V"
- note added: "from what i could tell a mosfet is built into the chip which is why the schematic has none"
- note added: "i couldn't quite figure out all the pins..."
- note removed: "V_out"
