File: lv/lv-onb-project/joshua-gonzalez-kicad/joshua-gonzalez-kicad.kicad_sch (KiCad schematic)
At the start: 0 parts

Commit message: Final Really Late Submission
Parts:
- added C1, C2, C3, C5: 0.1μF, Package_SO:SOIC-8_3.9x4.9mm_P1.27mm, symbol Device:C
- added R1: 16562.5, symbol Device:R
- added R2: 8437.5, symbol Device:R
- added R3: 3835, symbol Device:R
- added R4: 6335, symbol Device:R
- added U1: 4071, symbol 4xxx:4071
- added U2, U3, U4: OP1177AR, Package_SO:SOIC-8_3.9x4.9mm_P1.27mm, symbol Amplifier_Operational:OP1177AR
Connections:
- new net: U1.3, U1.5
- new net +5V: C1.2, C2.2, C3.2, C5.2, R1.1, R3.1, U1.14 (VDD), U2.7 (V+), U3.7 (V+), U4.7 (V+)
- new net BSPD_Fault_High: U1.4
- new net Current_Sensor: U3.3 (+)
- new net Current_Short_HIGH: U1.6, U3.6
- new net Front_Brake_HIGH: U1.1, U2.6
- new net Front_Brake_Sensor: U2.3 (+)
- new net GND: C1.1, C2.1, C3.1, C5.1, R2.2, R4.2, U1.7 (VSS), U2.4 (V-), U3.4 (V-), U4.4 (V-)
- new net Hard_Breaking_Threshold: R1.2, R2.1, U2.2 (-), U4.2 (-)
- new net High_Current_Threshold: R3.2, R4.1, U3.2 (-)
- new net Rear_Brake_HIGH: U1.2, U4.6
- new net Rear_Brake_Sensor: U4.3 (+)
- no-connect marks 0 -> 1
Other:
- note added: "3.375 V"
- note added: "Alright so it's a pretty basic BSPD. It essentially only checks for hard braking from the front and rear brake sensors (which is measuring for 1500 psi on the brakes) and whether or not the tractive system current delivering 5KW to the motor, in which case it activates a fault. I didn't implement more than a couple things such as the relay/timer which would be cool if I wasn't way over the deadli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"
- note added: "OR Gate Power Supply"
